File: vehicle/mkv/hardware/sensing_controller/suspension_travel.sch (KiCad schematic (older format))
At the start: 2 parts

Commit message: Remove rescue lib
Parts:
- C1801: symbol sensing_controller-rescue:C_22uF-formula -> formula:C_22uF
- R1801: symbol sensing_controller-rescue:R_1K_0.1-formula -> formula:R_1K_0.1
Changed lines of the file:
@@
 $EndDescr
 $Comp
-L sensing_controller-rescue:R_1K_0.1-formula R1801
+L formula:R_1K_0.1 R1801
 U 1 1 60A40AD2
 P 5500 3700
@@
 $EndComp
 $Comp
-L sensing_controller-rescue:C_22uF-formula C1801
+L formula:C_22uF C1801
 U 1 1 60A40ADB
 P 5500 4150
