File: vehicle/mkv/hardware/lvbox/lv_board/lv_board.sch (KiCad schematic (older format))
At the start: 121 parts, among them IC1 ATMEGA16M1, J1 Ampseal_35_VT, J11 MicroFit_VT_4, J12 MM_M_VT_20, J2 Ampseal_14_VT, J3 CONN_02X03, J3 MicroFit_VT_4, J7 MM_M_VT_20, J8 UF_2_VT, J9 MM_M_VT_20, K1 G5Q-1A4-DC12, Q1 SSM3K333R, Q2 SSM3K333R, Q3 SSM3K333R, Q6 SSM3K333R, U1 RJ45_VT, U1 SN74LVC1G08, U101 TPS560430YF, U2 Fuse_Holder_Blade, U2 MCP6001, U3 CAN_Transceiver, U3 Fuse_Holder_Blade, U4 MCP6001, U5 SN74LVC1G02, U6 SN74LVC1G02, U7 MCP6001, U8 SN74LVC1G32, Y1 Crystal_SMD

Commit message: label updates
Parts:
- removed R11, R12, R13, R14, R15, R16, R17: R_10K, footprints:R_0805_OEM, symbol formula:R_10K
- removed R41, R42: R_200, footprints:R_0805_OEM, symbol formula:R_200
- added R3, R4: R_200, footprints:R_0805_OEM, symbol formula:R_200
- added R40, R41, R42, R43, R44, R45: R_10K, footprints:R_0805_OEM, symbol formula:R_10K
- renumbered C102 to C10, C10 to C11, C16 to C12, C103 to C13, C17 to C14, C9 to C15, C12 to C16, C13 to C17, C7 to C18, C11 to C19, C14 to C20, C15 to C5, C5 to C6, C6 to C7, C101 to C8, C8 to C9, COUT101 to COUT1, COUT102 to COUT2, COUT103 to COUT3, D2 to D10, D5 to D11, D4 to D14, D2 to D15, D1 to D2, D101 to D3, D102 to D4, D2 to D5, D4 to D6, D3 to D7, D103 to D8, D1 to D9, F101 to F1, J3 to J1, J11 to J2, J1 to J4, J2 to J5, J7 to J6, J8 to J7, J9 to J8, J12 to J9, L101 to L1, Q3 to Q2, Q2 to Q3, Q1 to Q4, Q6 to Q5, R9 to R10, R101 to R11, R21 to R12, R11 to R13, R22 to R14, R13 to R15, R23 to R16, R102 to R18, R18 to R19, R4 to R2, R6 to R20, R103 to R21, R10 to R22, R104 to R23, R105 to R24, R4 to R25, R5 to R26, R44 to R27, R45 to R28, R46 to R29, R24 to R30, R12 to R31, R10 to R32, R15 to R33, R16 to R34, R19 to R35, R2 to R36, R20 to R37, R33 to R38, R34 to R39, R3 to R5, R5 to R6, R6 to R7, R7 to R8, R8 to R9, TP3 to TP1, TP1 to TP2, TP1 to TP3, TP2 to TP4, TP3 to TP5, TP2 to TP6, U8 to U10, U2 to U11, U3 to U12, U1 to U2, U2 to U3, U101 to U4, U3 to U7, U4 to U8, U7 to U9
Connections:
- net 12V is gone; now on net +12V: D1.1 (K), J1.2, J2.1, J4.11, J4.15, J4.2, J4.20, J5.13, J5.2, J6.2, J8.2, J9.2, K1.5, TP3.1
- net BRAKE PRESSURE SENSE is gone; now on net BRAKE_PRESSURE_SENSE: J5.8
- net BRAKELIGHT LSD is gone; now on net BRAKELIGHT_LSD: J5.3
- net BSPD CURRENT SENSE is gone; now on net VCC: J5.6
- net BSPD_CURRENT_SENSE is gone; now on net VCC: IC1.32 ((PCINT17/CLKO/PSCIN0)PD1), R2.2, U2.1 (in)
- net CAN + is gone; now on net CAN+: J1.3, J2.3, J4.13, J4.21, J5.10, J6.3, J8.3, J9.3, U1.2 (CANH)
- net CAN - is gone; now on net CAN-: J1.4, J2.4, J4.14, J4.22, J5.11, J6.4, J8.4, J9.4, U1.1 (CANL)
- net COOLING PUMP LSD is gone; now on net PUMP_RELAY_READ: J4.31
- net EXTRA TEMP 1 - is gone; now on net GND: J4.4
- net EXTRA TEMP 2 - is gone; now on net GND: J4.6
- net EXTRA TEMP 3 - is gone; now on net GND: J4.8
- net EXTRA TEMP 4 - is gone; now on net GND: J4.10
- net MC TEMP - is gone; now on net GND: J4.35
- net MOTOR TEMP - is gone; now on net GND: J4.33
- net RADIATOR TEMP - is gone; now on net GND: J4.19
- net RJ45 LED G is gone; now on net RJ45_LED_G: U1.12 (LED_2)
- net RJ45 LED O is gone; now on net RJ45_LED_O: U1.10 (LED_1)
- net GND: no longer IC1.13 ((PCINT21/ADC2/ACMP2)PD5), IC1.14 ((PCINT22/ADC3/INT0/ACMPN2)PD6), IC1.16 ((PCINT2/ADC5/INT1/ACMPN0)PB2), IC1.17 ((PCINT12/ADC8/ACMPN3/AMP1-)PC4), IC1.26 ((PCINT5/ADC6/INT2/ACMPN1/AMP2-)PB5), IC1.27 ((PCINT6/ADC7/PSCOUT1B)PB6), IC1.28 ((PCINT7/ADC4/SCK/PSCOUT0B)PB7)
- net RJ45_LED_G: now also R3.1
- net RJ45_LED_O: now also R4.2
- net VCC: now also R40.1, R41.1, R42.1, R43.1, R44.1, R45.1
- net at IC1.9 ((PCINT1/MOSI/PSCOUT2B)PB1): now also R4.1
- net at IC1.8 ((PCINT0/MISO/PSCOUT2A)PB0): now also R3.2
- net BRAKE PRESSURE + renamed BRAKE_PRESSURE+
- net BRAKE PRESSURE - renamed BRAKE_PRESSURE-
- net BSPD TEST SWITCH + renamed BSPD_TEST_SWITCH+
- net BSPD TEST SWITCH - renamed BSPD_TEST_SWITCH-
- net EXTRA TEMP 1 + renamed EXTRA_TEMP_1
- net EXTRA_TEMP_1: now also IC1.16 ((PCINT2/ADC5/INT1/ACMPN0)PB2), R40.2
- net EXTRA TEMP 2 + renamed EXTRA_TEMP_2
- net EXTRA_TEMP_2: now also IC1.13 ((PCINT21/ADC2/ACMP2)PD5), R43.2
- net EXTRA TEMP 3 + renamed EXTRA_TEMP_3
- net EXTRA_TEMP_3: now also IC1.14 ((PCINT22/ADC3/INT0/ACMPN2)PD6), R45.2
- net EXTRA TEMP 4 + renamed EXTRA_TEMP_4
- net EXTRA_TEMP_4: now also IC1.17 ((PCINT12/ADC8/ACMPN3/AMP1-)PC4), R42.2
- net MC TEMP + renamed MC_TEMP_READ
- net MC_TEMP_READ: now also IC1.26 ((PCINT5/ADC6/INT2/ACMPN1/AMP2-)PB5), R41.2
- net MOTOR TEMP + renamed MOTOR_TEMP_READ
- net MOTOR_TEMP_READ: now also IC1.27 ((PCINT6/ADC7/PSCOUT1B)PB6), R44.2
- net RADIATOR TEMP + renamed RADIATOR_READ
- net RADIATOR_READ: now also IC1.28 ((PCINT7/ADC4/SCK/PSCOUT0B)PB7)
Other:
- note added: "CONNECTORS\n"
- note added: "fix spaces!"
- note removed: "COOLING EXTRA SENSING?\n"
- note removed: "Extra Temp 1?\n"
- note removed: "Extra Temp 2?\n"
- note removed: "Extra Temp 3?\n"
- note removed: "Extra Temp 4?\n"
- note removed: "MC Temp?"
- note removed: "Motor Temp?\n"
- note removed: "Radiator Temp?\n"
- note removed: "Shutdown\n\n"
- moved on the sheet: D14, D15, J4, J5, J6, J7, J8, J9, TP1, U11, U12
