File: vehicle/mkv/hardware/lvbox/lvbms/lv_bms/lv_bms_2.sch (KiCad schematic (older format))
At the start: 121 parts, among them J1 CONN_02X03, J10 NanoFit_RA_TH_04, J2 NanoFit_RA_TH_06, J3 NanoFit_RA_TH_02, J5 NanoFit_RA_TH_02, J6 NanoFit_RA_TH_02, J7 NanoFit_RA_TH_02, J8 NanoFit_RA_TH_02, J9 NanoFit_RA_TH_02, Q1 NSS1C201MZ4, Q2 SQM110P06, Q3 BSS138, Q4 BSS138, Q5 SQM110P06, Q6 BSS138, U1 MCP2561-E_SN, U10 ACHS-7124, U11 redcube-7461057, U2 ATMEGA16M1, U3 LTC6810HG-2, U4 LT3066IMSE-5, U5 LT1017IS8, U6 R_500, U7 R_500, U8 R_500, U9 redcube-7461057, Y1 Crystal_SMD

Commit message: layout first pass gd mfs
Parts:
- removed F1: 0685P9500-01, footprints:Fuse_1206, symbol formula:0685P9500-01
- removed F101: F_500mA_16V, footprints:Fuse_1210, symbol formula:F_500mA_16V
- removed J10: NanoFit_RA_TH_04, footprints:NanoFit_RA_4, symbol formula:NanoFit_RA_TH_04
- removed J2: NanoFit_RA_TH_06, footprints:NanoFit_RA_6, symbol formula:NanoFit_RA_TH_06
- removed J3, J5, J6, J7, J8, J9: NanoFit_RA_TH_02, footprints:NanoFit_Molex_1x02x2.50mm_Angled_OEM, symbol formula:NanoFit_RA_TH_02
- removed Q3, Q4: BSS138, Package_TO_SOT_SMD:SOT-23, symbol Transistor_FET:BSS138
- removed R29, R31: R_0_2512, footprints:R_2512_OEM, symbol formula:R_0_2512
- removed R32, R33, R35, R36: R_200, footprints:R_0805_OEM, symbol formula:R_200
- removed R34: R_10K, footprints:R_0805_OEM, symbol formula:R_10K
- removed R4, R5, R6, R7, R8: R_30_6W_1%, footprints:356030RFT, symbol formula:R_30_6W_1%
- removed U6, U7, U8: R_500, footprints:R_0805_OEM, symbol formula:R_500
- added D5: LED_0805_Red, footprints:LED_0805_OEM, symbol formula:LED_0805_Red
- added F1: F_500mA_60V, footprints:Fuse_1812_4532Metric, symbol formula:F_500mA_60V
- added F2: F_50A_32V, footprints:Fuse_1206, symbol formula:F_50A_32V
- added J2: NanoFit_RA_SMT_04, footprints:NanoFit_RA_SMT_04, symbol formula:NanoFit_RA_SMT_04
- added J3, J4, J5, J6, J7, J9: NanoFit_RA_SMT_02, footprints:NanoFit_RA_SMT_02, symbol formula:NanoFit_RA_SMT_02
- added J8: NanoFit_RA_SMT_06_A, footprints:NanoFit_RA_SMT_06, symbol formula:NanoFit_RA_SMT_06_A
- added Q3, Q4: SSM3K333R, footprints:SOT-23F, symbol formula:SSM3K333R
- added R29, R45, R46: R_500, footprints:R_0805_OEM, symbol formula:R_500
- added R32, R34, R35, R36, R43: R_499, footprints:R_0805_OEM, symbol formula:R_499
- added R33: R_5K, footprints:R_0805_OEM, symbol formula:R_5K
- added R4, R5, R6, R7, R8: R_15_1W_.5%, footprints:Fuse_1206, symbol formula:R_15_1W_.5%
- added R44: R_0, footprints:R_0603_1608Metric, symbol formula:R_0
- added TP18, TP19: Test_Point_SMD, TestPoint:TestPoint_Pad_D1.5mm, symbol formula:Test_Point_SMD
- added TP20: Test_Point_SMD, footprints:Test_Point_SMD, symbol formula:Test_Point_SMD
- C10, C15, C6, C7, C8, C9: footprint footprints:C_1206_OEM -> footprints:C_0805_OEM
- R19: footprint footprints:R_2010_Vishay -> footprints:R_0805_OEM
- TP1, TP10, TP11, TP12, TP13, TP14, TP15, TP17, TP2, TP3, TP4, TP5, TP6, TP7, TP8, TP9: footprint footprints:Test_Point_SMD -> TestPoint:TestPoint_Pad_D1.5mm
Connections:
- net labels added: CAN_N, CAN_P
- net labels removed: BATTERY_SIDE_DIV_SIG, CAN+, CAN-, SHUNT_LOAD_SIDE
- wire segments 269 -> 272
- no-connect marks 15 -> 14
Other:
- note added: "10K NTC thermistor \nresistor dividers, \nonly powered on \nafter Wakeup - \nexpect 2.5V @ 25C"
- note added: "10V - 16.8V \nInput Voltage"
- note added: "5 individual nanofit connectors for thermistors \nto be distributed around the edges of the PCB\nhttps://www.digikey.com/en/products/detail\n/epcos-tdk/B57861S0103F040/739889"
- note added: "Comparator logic chart \n\n| | No Load | Charging | Discharging | FAULT |\n|--------|------|------|---------|-----|\n| comp_1_out | 1 | 1 | 0 | 0 |\n| comp_2_out | 1 | 0 | 1 | 0 |\n\nThe outputs of both comparators are fed into \nLOW Level Triggered External interrupts on the Atemga\nwhere C1 LOW indicates Discharge state & C2 LOW \nindicates Charge state. \n\nBoth C1 and C2 low triggers a WAKEUP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"
- note added: "Linreg will dissipate 2.35W \nnominally continuously w/\nsystem in ON state. \nWith 400mm Cu, an Rth J-A \nof 37C/W, Junction temp \n=86.95C"
- note added: "Optional Battery (-)\nGND Power Lead \nwire connection"
- note added: "The high current path on this \nPCB will see 20A continuous, \n30A peak for 1 hour with the \ncooling pack, and 5A continuous \nwith the GLV pack. Our high \ncurrent path features a current \nsensor, bidirectional load switch, \nand fuse. \n\nThe fuse and current sensor are \ndifferent between GLV system \nand cooling pack system. \n\nThe bidirectional load switch was \ntested with the LV BMS Tes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"
- note removed: "10K thermistor \nresistor dividers, \nonly powered on \nafter Wakeup"
- note removed: "6 individual nanofit connectors for thermistors \nto be distributed around the edges of the PCB\nhttps://www.digikey.com/en/products/detail\n/epcos-tdk/B57861S0103F040/739889"
- note removed: "BATT_4 Jumper\n"
- note removed: "Comparator logic chart \n+--------+------+-----+---------+\n| | No Load | Charging | Discharging |\n+--------+------+-----+---------+\n| COMP_1_OUT | 1 | 1 | 0 |\n+--------+------+-----+---------+\n| COMP_2_OUT | 1 | 0 | 1 |\n+--------+------+-----+---------+\n\nThe outputs of both comparators are fed into \nLOW Level Triggered External interrupts on the Atemga\nwhere C1 LOW indicates Discharge s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"
- note removed: "The high current path on this \nPCB will see 20A continuous, \n30A peak for 1 hour with the \ncooling pack, and 5A continuous \nwith the GLV pack. Our high \ncurrent path features a current \nsensor, bidirectional load switch, \nand fuse. \n\nThe fuse and current sensor are \nswappable between GLV system \nand cooling pack system. \n\nThe bidirectional load switch was \ntested with the LV BMS Tes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"
- moved on the sheet: C15, C19, R15, R16, R17, R21, R22, R23, R24, R25, R26, R27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

Commit message: layout rev2 completed
Parts:
- added Q7, Q8: SQM110P06, footprints:TO-263-3-TabPin2, symbol formula:SQM110P06
- added TP21, TP22, TP23, TP24, TP25, TP26, TP27, TP28: Test_Point_SMD, footprints:Test_Point_SMD, symbol formula:Test_Point_SMD
Connections:
- net GND: now also TP21.1, TP22.1
- net LOAD_SIDE_CURRENT_PATH: now also Q8.2 (D)
- net ON_STATE_CMPNTS_-: now also TP24.1, TP26.1, TP28.1
- net THERM_0_+: now also TP23.1
- net THERM_1_+: now also TP25.1
- net THERM_2_+: now also TP27.1
- net THERM_3_+: now also TP18.1
- net THERM_4_+: no longer TP18.1
- net at Q2.2 (D), U10.3 (IP-), U10.4 (IP-): now also Q7.2 (D)
- net at Q2.1 (G), Q5.1 (G), R40.2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: now also Q7.1 (G), Q8.1 (G)
- net at Q2.3 (S), Q5.3 (S), R40.1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: now also Q7.3 (S), Q8.3 (S)
Other:
- note added: "DNP\nFET"
- moved on the sheet: Q2, Q5, Q6, R38, R40, R41, TP13, TP6, U11
