File: vehicle/mkv/hardware/service_section_controller/air_control.sch (KiCad schematic (older format))
At the start: 25 parts, among them Q901 SSM3K333R, Q902 SSM3K333R

Commit message: incorporated feedback from dr
Parts:
- renumbered D902 to D901, D901 to D902, D904 to D903, D903 to D904, R902 to R901, R904 to R902, R901 to R903, R903 to R904, R907 to R905, R905 to R906, R908 to R907, R906 to R908
Changed lines of the file:
@@
 AIR CONTROL RELAY CIRCUITS
 $Comp
-L power:GND #PWR?
+L power:GND #PWR0904
 U 1 1 61065F69
 P 5850 5550
-F 0 "#PWR?" H 5850 5300 50  0001 C CNN
+F 0 "#PWR0904" H 5850 5300 50  0001 C CNN
 F 1 "GND" H 5855 5377 50  0000 C CNN
 F 2 "" H 5850 5550 50  0001 C CNN
@@
 $EndComp
 $Comp
-L formula:R_10K R906
+L formula:R_10K R908
 U 1 1 61065F72
 P 5850 4900
-F 0 "R906" V 5750 4850 50  0000 L CNN
+F 0 "R908" V 5750 4850 50  0000 L CNN
 F 1 "R_10K" V 5950 4800 50  0000 L CNN
 F 2 "footprints:R_0805_OEM" H 5780 4900 50  0001 C CNN
@@
 $EndComp
 $Comp
-L formula:LED_0805 D903
+L formula:LED_0805 D904
 U 1 1 61065F7B
 P 5300 5200
-F 0 "D903" V 5300 5450 50  0000 R CNN
+F 0 "D904" V 5300 5450 50  0000 R CNN
 F 1 "LED_0805" V 5200 5600 50  0000 R CNN
 F 2 "footprints:LED_0805_OEM" H 5200 5200 50  0001 C CNN
@@
 $EndComp
 $Comp
-L formula:R_200 R905
+L formula:R_200 R906
 U 1 1 61065F84
 P 5300 4800
-F 0 "R905" H 5050 4750 50  0000 L CNN
+F 0 "R906" H 5050 4750 50  0000 L CNN
 F 1 "R_200" H 5000 4850 50  0000 L CNN
 F 2 "footprints:R_0805_OEM" H 5230 4800 50  0001 C CNN
@@
 Wire Wire Line
 	5300 4600 5600 4600
-Wire Wire Line
-	5800 4000 5350 4000
-$Comp
-L power:GND #PWR?
+$Comp
+L power:GND #PWR0902
 U 1 1 61065F96
 P 3400 5550
-F 0 "#PWR?" H 3400 5300 50  0001 C CNN
+F 0 "#PWR0902" H 3400 5300 50  0001 C CNN
 F 1 "GND" H 3405 5377 50  0000 C CNN
 F 2 "" H 3400 5550 50  0001 C CNN
@@
 	2900 4650 3150 4650
 $Comp
-L formula:R_200 R901
+L formula:R_200 R903
 U 1 1 61065FAA
 P 2900 4850
-F 0 "R901" H 2650 4800 50  0000 L CNN
+F 0 "R903" H 2650 4800 50  0000 L CNN
 F 1 "R_200" H 2600 4900 50  0000 L CNN
 F 2 "footprints:R_0805_OEM" H 2830 4850 50  0001 C CNN
@@
 $EndComp
 $Comp
-L formula:R_10K R903
+L formula:R_10K R904
 U 1 1 61065FB3
 P 3400 5050
-F 0 "R903" H 3450 5100 50  0000 L CNN
+F 0 "R904" H 3450 5100 50  0000 L CNN
 F 1 "R_10K" H 3450 5000 50  0000 L CNN
 F 2 "footprints:R_0805_OEM" H 3330 5050 50  0001 C CNN
@@
 Wire Wire Line
 	3650 4000 2950 4000
-Text Notes 4950 3800 0    98   ~ 0
+Text Notes 5000 3650 0    98   ~ 0
 Air+ Weld Detection
 $Comp
-L power:GND #PWR?
+L power:GND #PWR0906
 U 1 1 61066001
 P 6350 3100
-F 0 "#PWR?" H 6350 2850 50  0001 C CNN
+F 0 "#PWR0906" H 6350 2850 50  0001 C CNN
 F 1 "GND" H 6355 2927 50  0000 C CNN
 F 2 "" H 6350 3100 50  0001 C CNN
@@
 	6350 2350 6350 3100
 $Comp
-L formula:LED_0805 D904
+L formula:LED_0805 D903
 U 1 1 6106600B
 P 5200 2850
-F 0 "D904" V 5150 2800 50  0000 R CNN
+F 0 "D903" V 5150 2800 50  0000 R CNN
 F 1 "LED_0805" V 5250 2800 50  0000 R CNN
 F 2 "footprints:LED_0805_OEM" H 5100 2850 50  0001 C CNN
@@
 $EndComp
 $Comp
-L formula:R_10K R908
+L formula:R_10K R907
 U 1 1 61066016
 P 5650 2600
-F 0 "R908" H 5720 2646 50  0000 L CNN
+F 0 "R907" H 5720 2646 50  0000 L CNN
 F 1 "R_10K" H 5720 2555 50  0000 L CNN
 F 2 "footprints:R_0805_OEM" H 5580 2600 50  0001 C CNN
@@
 $EndComp
 $Comp
-L formula:R_200 R907
+L formula:R_200 R905
 U 1 1 61066021
 P 5200 2400
-F 0 "R907" H 5250 2350 50  0000 L CNN
+F 0 "R905" H 5250 2350 50  0000 L CNN
 F 1 "R_200" H 5250 2450 50  0000 L CNN
 F 2 "footprints:R_0805_OEM" H 5130 2400 50  0001 C CNN
@@
 $EndComp
 $Comp
-L power:GND #PWR?
+L power:GND #PWR0901
 U 1 1 61066035
 P 3150 3000
-F 0 "#PWR?" H 3150 2750 50  0001 C CNN
+F 0 "#PWR0901" H 3150 2750 50  0001 C CNN
 F 1 "GND" H 3155 2827 50  0000 C CNN
 F 2 "" H 3150 3000 50  0001 C CNN
@@
 $EndComp
 $Comp
-L formula:R_200 R902
+L formula:R_200 R901
 U 1 1 61066040
 P 2050 2400
-F 0 "R902" H 1800 2350 50  0000 L CNN
+F 0 "R901" H 1800 2350 50  0000 L CNN
 F 1 "R_200" H 1750 2450 50  0000 L CNN
 F 2 "footprints:R_0805_OEM" H 1980 2400 50  0001 C CNN
@@
 $EndComp
 $Comp
-L formula:LED_0805 D902
+L formula:LED_0805 D901
 U 1 1 61066049
 P 2050 2800
-F 0 "D902" V 2050 3050 50  0000 R CNN
+F 0 "D901" V 2050 3050 50  0000 R CNN
 F 1 "LED_0805" V 1950 3200 50  0000 R CNN
 F 2 "footprints:LED_0805_OEM" H 1950 2800 50  0001 C CNN
@@
 Wire Wire Line
 	5300 5450 5850 5450
-Text Notes 2850 3800 0    98   ~ 0
+Text Notes 2900 3700 0    98   ~ 0
 Air- Weld Detection
 $Comp
-L formula:R_10K R904
+L formula:R_10K R902
 U 1 1 61066090
 P 2400 2550
-F 0 "R904" H 2470 2596 50  0000 L CNN
+F 0 "R902" H 2470 2596 50  0000 L CNN
 F 1 "R_10K" H 2470 2505 50  0000 L CNN
 F 2 "footprints:R_0805_OEM" H 2330 2550 50  0001 C CNN
@@
 	5600 4250 5600 4600
 Connection ~ 5600 4600
-Text GLabel 3650 4000 2    50   Input ~ 0
-5V_AIR_CONTROL
-Text GLabel 5800 4000 2    50   Input ~ 0
-5V_AIR_CONTROL
 Connection ~ 10100 2700
 Wire Wire Line
 	10100 2700 10100 2850
 $Comp
-L power:GND #PWR?
+L power:GND #PWR0907
 U 1 1 61065FC3
 P 10100 2850
-F 0 "#PWR?" H 10100 2600 50  0001 C CNN
+F 0 "#PWR0907" H 10100 2600 50  0001 C CNN
 F 1 "GND" H 10105 2677 50  0000 C CNN
 F 2 "" H 10100 2850 50  0001 C CNN
@@
 	3400 5200 3400 5450
 $Comp
-L formula:LED_0805 D901
+L formula:LED_0805 D902
 U 1 1 61065FA0
 P 2900 5200
-F 0 "D901" V 2900 5450 50  0000 R CNN
+F 0 "D902" V 2900 5450 50  0000 R CNN
 F 1 "LED_0805" V 2800 5600 50  0000 R CNN
 F 2 "footprints:LED_0805_OEM" H 2800 5200 50  0001 C CNN
@@
 Wire Wire Line
 	5950 4600 6100 4600
+Wire Wire Line
+	5350 4000 6050 4000
+Text GLabel 6050 4000 2    50   Input ~ 0
++5V_AIR_CONTROL
+Text GLabel 3650 4000 2    50   Input ~ 0
++5V_AIR_CONTROL
 $EndSCHEMATC
