File: vehicle/gokart/hardware/bms_core/bms_core.kicad_pcb (KiCad board)
At the start: 2 copper layers, 59.2 x 59.2 mm, 65 parts, among them J1 CONN_02X03, J2 NanoFit_RA_TH_02, J3 MicroFit_RA_4, J4 NanoFit_RA_TH_02, J5 MicroFit_RA_4, J6 MicroFit_RA_4, J7 MicroFit_RA_4, Q1 SSM3K333R, Q2 SSM3K333R, Q3 SSM3K333R, Q4 SSM3J334R, Q5 SSM3K333R, T1 T_LAN_SM91501ALE, U1 MCP2561-E_SN, U2 ATMEGA16M1, U3 AP7370, U4 LTC6820HMS, Y1 Crystal_SMD

Commit message: chore: migrate projects to kicad 6
Other:
- net class Default removed
