File: vehicle/mkv/hardware/service_section/peripheral/bms_peripheral.kicad_pcb (KiCad board)
At the start: 4 copper layers, 50 x 287 mm, 133 parts, among them J1 MM_F_VT_12, J2 MM_F_VT_10, J3 MM_F_VT_16, J4 MM_F_VT_12, J5 MM_M_VT_12, J6 MicroFit_RA_V_2_SMD, J7 MicroFit_RA_V_2_SMD, Q1 NSS1C201MZ4, Q2 NSS1C201MZ4, T1 T_LAN_SM91501ALE, T2 T_LAN_SM91501ALE, U1 LTC6811-1, U2 LTC6811-1, U3 24AA01, U4 MCP6001T-I-LT, U5 LTC1380IGN, U6 LTC1380IGN, U7 LTC1380IGN, U8 MCP6001T-I-LT

Commit message: chore: migrate projects to kicad 6
Connections:
- net /~DIS~1 renamed /~{DIS}1
- net /~DIS~2 renamed /~{DIS}2
- net /~DIS~3 renamed /~{DIS}3
- net /~DIS~4 renamed /~{DIS}4
- net /~DIS~6 renamed /~{DIS}6
- net /~DIS~7 renamed /~{DIS}7
- net /~DIS~8 renamed /~{DIS}8
- net /~DIS~9 renamed /~{DIS}9
Other:
- net class Default removed
