File: projects/hitl/hardware/primary_board/hitl-primary.kicad_pcb (KiCad board)
At the start: 4 copper layers, 108 x 79.7 mm, 132 parts, among them J1 USB-Micro-1981568-1, J10 CONN_01X03, J11 CONN_01X03, J12 CONN_01X03, J13 CONN_01x02, J14 SSW-122-01-G-D, J15 CONN_01x02, J16 CONN_01X03, J17 CONN_01X03, J18 CONN_01X03, J19 CONN_01X03, J2 Barrel_jack, J20 CONN_01X03, J21 Screw_Terminal_01x03, J3 MM_F_VT_08_SM, J4 MM_F_VT_08_SM, J6 CONN_01x02, J7 CONN_01X03, J8 CONN_01X03, J9 CONN_01X03, Q1 SSM3K333R, Q2 SSM3K333R, Q3 SSM3K333R, Q4 SSM3K333R, SW1 SW_SPST, U1 PCA9517, U2 FT4222H, U4 AD5675, U5 MAX7300AAXT, U6 AD7091R-5BRUZ, U7 MCP6001, U8 74HCT4051D, U9 LT3045, Y1 Crystal_12MHz

Commit message: Add QR Code
Parts:
- added G***: LOGO, footprints:Small_OE_Logo, B.Cu at (127.3, 43.3)
- added QR*****: Scan for docs, qr.olinelectricmotorsports.com/hw/hitl/1.1, B.Cu at (83.6, 61.9)
- added kibuzzard-632DCC16: G***, kibuzzard-632DCC16, B.Cu at (153.5, 38.5)
Other:
- board text added: "Corey Cochran-Lepiz Alex Wenstrup Jack Greenberg"
- board text added: "Rev 1.1"
