File: examples/m.2_example/daughter/m.2_daughter.kicad_sch (KiCad schematic)
At the start: 33 parts, among them J1 CONN_02X03, J2 M.2_BoardEdge, K1 G5Q-1A4-DC12, Q1 SSM3K333R, Q2 SSM3K333R, Q3 SSM3K333R, U1 MCP2561-E_SN, U2 ATMEGA16M1, Y1 Crystal_SMD

Commit message: feat: arduino-esque motherboard
Parts:
- J2: symbol formula:M.2_BoardEdge -> formula:Automotive_M.2_Edge_Connector
Changed lines of the file:
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@@
     (pin "2")
   )
-  (symbol (lib_id "formula:M.2_BoardEdge") (at 316.23 149.86 0) (unit 1)
+  (symbol (lib_id "formula:Automotive_M.2_Edge_Connector") (at 316.23 149.86 0) (unit 1)
     (in_bom yes) (on_board yes) (fields_autoplaced)
     (property "Reference" "J2" (id 0) (at 316.23 100.584 0)
