File: vehicle/mkvi/rkh/bspd.kicad_sch (KiCad schematic)
At the start: 7 parts, among them J601 Automotive_M.2, SW601 SW_SPST, U601 TMUX1247DCKR

Commit message: Checkpoint
Parts:
- removed D601: LED, symbol Device:LED
- removed SW601: SW_SPST, symbol Switch:SW_SPST
- added D601: LED_0805, footprints:LED_0805_OEM, symbol formula:LED_0805
- U601: footprint SOT-SC70_DCK_6_TEX -> footprints:TMUX1247DCKR
Connections:
- net BRAKELIGHT_LSD: now also D601.1 (K)
- net at R601.2: now also D601.2 (A)
- net AMUX_SEL renamed HITL_BRKPRES_SEL
Other:
- note removed: "In case BSPD doesn't work"
Changed lines of the file:
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@@
 (kicad_sch (version 20211123) (generator eeschema)
   (paper "A4")
-  (junction (at 95.25 107.95) (diameter 0) (color 0 0 0 0)
-  )
-  (junction (at 95.25 97.79) (diameter 0) (color 0 0 0 0)
-  )
   (junction (at 135.89 53.34) (diameter 0) (color 0 0 0 0)
   )
@@
     (stroke (width 0) (type default) (color 0 0 0 0))
   )
-  (wire (pts (xy 86.36 107.95) (xy 95.25 107.95))
-    (stroke (width 0) (type default) (color 0 0 0 0))
-  )
   (wire (pts (xy 54.61 44.45) (xy 55.88 44.45))
     (stroke (width 0) (type default) (color 0 0 0 0))
@@
     (stroke (width 0) (type default) (color 0 0 0 0))
   )
-  (wire (pts (xy 109.22 107.95) (xy 109.22 104.14))
-    (stroke (width 0) (type default) (color 0 0 0 0))
-  )
   (wire (pts (xy 135.89 88.9) (xy 135.89 90.17))
     (stroke (width 0) (type default) (color 0 0 0 0))
@@
     (stroke (width 0) (type default) (color 0 0 0 0))
   )
-  (wire (pts (xy 95.25 107.95) (xy 109.22 107.95))
-    (stroke (width 0) (type default) (color 0 0 0 0))
-  )
   (wire (pts (xy 135.89 53.34) (xy 135.89 55.88))
     (stroke (width 0) (type default) (color 0 0 0 0))
   )
-  (wire (pts (xy 109.22 97.79) (xy 95.25 97.79))
-    (stroke (width 0) (type default) (color 0 0 0 0))
-  )
-  (wire (pts (xy 109.22 101.6) (xy 109.22 97.79))
-    (stroke (width 0) (type default) (color 0 0 0 0))
-  )
   (wire (pts (xy 135.89 50.8) (xy 135.89 53.34))
     (stroke (width 0) (type default) (color 0 0 0 0))
   )
-  (wire (pts (xy 95.25 97.79) (xy 86.36 97.79))
-    (stroke (width 0) (type default) (color 0 0 0 0))
-  )
   (wire (pts (xy 127 69.85) (xy 135.89 69.85))
     (stroke (width 0) (type default) (color 0 0 0 0))
@@
     (effects (font (size 1.27 1.27)) (justify left bottom))
   )
-  (text "In case BSPD doesn't work" (at 87.63 111.76 0)
-    (effects (font (size 1.27 1.27)) (justify left bottom))
-  )
   (label "GND" (at 135.89 93.98 180)
     (effects (font (size 1.27 1.27)) (justify right bottom))
@@
     (effects (font (size 1.27 1.27)) (justify left bottom))
   )
-  (global_label "AMUX_SEL" (shape input) (at 55.88 55.88 180) (fields_autoplaced)
-    (effects (font (size 1.27 1.27)) (justify right))
-    (property "Intersheet References" "${INTERSHEET_REFS}" (id 0) (at 44.0326 55.8006 0)
-      (effects (font (size 1.27 1.27)) (justify right) hide)
-    )
-  )
   (hierarchical_label "BRAKE_PRESSURE_SENSE" (shape input) (at 135.89 81.28 180)
     (effects (font (size 1.27 1.27)) (justify right))
@@
     (effects (font (size 1.27 1.27)) (justify right))
   )
-  (hierarchical_label "SHDN_TO_BSPD" (shape input) (at 86.36 97.79 180)
-    (effects (font (size 1.27 1.27)) (justify right))
-  )
-  (hierarchical_label "SHDN_SENSE_BSPD" (shape output) (at 123.19 118.11 180)
+  (hierarchical_label "SHDN_SENSE_BSPD" (shape output) (at 107.95 111.76 180)
     (effects (font (size 1.27 1.27)) (justify right))
   )
@@
     (effects (font (size 1.27 1.27)) (justify right))
   )
-  (hierarchical_label "SHDN_FROM_BSPD" (shape input) (at 86.36 107.95 180)
+  (hierarchical_label "HITL_BRKPRES_SEL" (shape input) (at 55.88 55.88 180)
     (effects (font (size 1.27 1.27)) (justify right))
   )
@@
     (pin "P40")
   )
+  (symbol (lib_id "formula:LED_0805") (at 201.93 105.41 90) (unit 1)
+    (in_bom yes) (on_board yes)
+    (property "Reference" "D601" (id 0) (at 198.12 104.14 90))
+    (property "Value" "LED_0805" (id 1) (at 194.31 106.68 90))
+    (property "Footprint" "footprints:LED_0805_OEM" (id 2) (at 201.93 107.95 0)
+      (effects (font (size 1.27 1.27)) hide)
+    )
+    (property "Datasheet" "http://www.osram-os.com/Graphics/XPic9/00078860_0.pdf" (id 3) (at 199.39 105.41 0)
+      (effects (font (size 1.27 1.27)) hide)
+    )
+    (property "MFN" "DK" (id 4) (at 201.93 105.41 0)
+      (effects (font (size 1.524 1.524)) hide)
+    )
+    (property "MPN" "475-1410-1-ND" (id 5) (at 201.93 105.41 0)
+      (effects (font (size 1.524 1.524)) hide)
+    )
+    (property "PurchasingLink" "https://www.digikey.com/products/en?keywords=475-1410-1-ND" (id 6) (at 189.23 95.25 0)
+      (effects (font (size 1.524 1.524)) hide)
+    )
+    (pin "1")
+    (pin "2")
+  )
   (symbol (lib_id "formula:C_1uF") (at 52.07 41.91 90) (unit 1)
     (in_bom yes) (on_board yes)
@@
     (pin "2")
   )
-  (symbol (lib_id "Device:LED") (at 201.93 105.41 90) (unit 1)
-    (in_bom yes) (on_board yes) (fields_autoplaced)
-    (property "Reference" "D601" (id 0) (at 205.74 105.7274 90)
-      (effects (font (size 1.27 1.27)) (justify right))
-    )
-    (property "Value" "LED" (id 1) (at 205.74 108.2674 90)
-      (effects (font (size 1.27 1.27)) (justify right))
-    )
-    (property "Footprint" "" (id 2) (at 201.93 105.41 0)
-      (effects (font (size 1.27 1.27)) hide)
-    )
-    (property "Datasheet" "~" (id 3) (at 201.93 105.41 0)
-      (effects (font (size 1.27 1.27)) hide)
-    )
-    (pin "1")
-    (pin "2")
-  )
   (symbol (lib_id "formula:TMUX1247DCKR") (at 66.04 49.53 0) (unit 1)
     (in_bom yes) (on_board yes) (fields_autoplaced)
@@
       (effects (font (size 1.524 1.524)))
     )
-    (property "Footprint" "SOT-SC70_DCK_6_TEX" (id 2) (at 111.125 41.91 0)
+    (property "Footprint" "footprints:TMUX1247DCKR" (id 2) (at 111.125 41.91 0)
       (effects (font (size 1.524 1.524)) hide)
     )
@@
     (pin "1")
   )
-  (symbol (lib_id "Switch:SW_SPST") (at 95.25 102.87 90) (unit 1)
-    (in_bom yes) (on_board yes)
-    (property "Reference" "SW601" (id 0) (at 96.52 101.5999 90)
-      (effects (font (size 1.27 1.27)) (justify right))
-    )
-    (property "Value" "SW_SPST" (id 1) (at 96.52 104.1399 90)
-      (effects (font (size 1.27 1.27)) (justify right))
-    )
-    (property "Footprint" "" (id 2) (at 95.25 102.87 0)
-      (effects (font (size 1.27 1.27)) hide)
-    )
-    (property "Datasheet" "~" (id 3) (at 95.25 102.87 0)
-      (effects (font (size 1.27 1.27)) hide)
-    )
-    (pin "1")
-    (pin "2")
-  )
   (symbol (lib_id "power:GND") (at 76.2 58.42 0) (unit 1)

Commit message: Add potentiometer footprint
Parts:
- RV601: footprint (none) -> footprints:PTV09A4020FB103
Changed lines of the file:
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@@
     (property "Reference" "RV601" (id 0) (at 63.5 76.2 0))
     (property "Value" "R_Potentiometer" (id 1) (at 67.31 66.04 0))
-    (property "Footprint" "" (id 2) (at 67.31 76.2 0)
+    (property "Footprint" "footprints:PTV09A4020FB103" (id 2) (at 67.31 76.2 0)
       (effects (font (size 1.27 1.27)) hide)
     )

Commit message: Checkpoint
Connections:
- net BRAKE_PRESSURE_N is gone; now on net GND: RV601.3
- net BRAKE_PRESSURE_P is gone; now on net +5V: RV601.1
- net BRAKE_PRESSURE_POT: now also U601.3 (S1); no longer U601.1 (S2)
- net HITL_BRAKE_PRESSURE: now also U601.1 (S2); no longer U601.3 (S1)
Other:
- moved on the sheet: RV601
Changed lines of the file:
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@@
-    (stroke (width 0) (type default) (color 0 0 0 0))
-  )
-  (wire (pts (xy 64.77 72.39) (xy 67.31 72.39))
-    (stroke (width 0) (type default) (color 0 0 0 0))
-  )
-  (wire (pts (xy 64.77 80.01) (xy 67.31 80.01))
     (stroke (width 0) (type default) (color 0 0 0 0))
   )
@@
     (stroke (width 0) (type default) (color 0 0 0 0))
   )
+  (wire (pts (xy 58.42 86.36) (xy 58.42 85.09))
+    (stroke (width 0) (type default) (color 0 0 0 0))
+  )
   (wire (pts (xy 135.89 50.8) (xy 135.89 53.34))
     (stroke (width 0) (type default) (color 0 0 0 0))
   )
+  (wire (pts (xy 58.42 76.2) (xy 58.42 77.47))
+    (stroke (width 0) (type default) (color 0 0 0 0))
+  )
   (wire (pts (xy 127 69.85) (xy 135.89 69.85))
     (stroke (width 0) (type default) (color 0 0 0 0))
@@
     (stroke (width 0) (type default) (color 0 0 0 0))
   )
+  (wire (pts (xy 64.77 81.28) (xy 62.23 81.28))
+    (stroke (width 0) (type default) (color 0 0 0 0))
+  )
   (wire (pts (xy 135.89 90.17) (xy 135.89 91.44))
     (stroke (width 0) (type default) (color 0 0 0 0))
@@
     (stroke (width 0) (type default) (color 0 0 0 0))
   )
-  (text "Brake Pressure" (at 61.595 84.455 0)
+  (text "Brake Pressure" (at 52.07 95.25 0)
     (effects (font (size 1.27 1.27)) (justify left bottom))
   )
@@
     (effects (font (size 1.27 1.27)) (justify left bottom))
   )
-  (label "BRAKE_PRESSURE_POT" (at 55.88 48.26 180)
+  (label "BRAKE_PRESSURE_POT" (at 55.88 50.8 180)
     (effects (font (size 1.27 1.27)) (justify right bottom))
   )
@@
     (effects (font (size 1.27 1.27)) (justify right bottom))
   )
+  (label "BRAKE_PRESSURE_SENSE" (at 135.89 81.28 180)
+    (effects (font (size 1.27 1.27)) (justify right bottom))
+  )
   (label "BRAKELIGHT_+" (at 201.93 90.17 0)
     (effects (font (size 1.27 1.27)) (justify left bottom))
@@
     (effects (font (size 1.27 1.27)) (justify right bottom))
   )
-  (label "BRAKE_PRESSURE_N" (at 64.77 80.01 180)
-    (effects (font (size 1.27 1.27)) (justify right bottom))
-  )
   (label "GND" (at 135.89 106.68 180)
     (effects (font (size 1.27 1.27)) (justify right bottom))
@@
     (effects (font (size 1.27 1.27)) (justify left bottom))
   )
-  (label "BRAKE_PRESSURE_P" (at 64.77 72.39 180)
-    (effects (font (size 1.27 1.27)) (justify right bottom))
-  )
-  (label "BRAKE_PRESSURE_SENSE" (at 71.12 76.2 0)
-    (effects (font (size 1.27 1.27)) (justify left bottom))
-  )
-  (hierarchical_label "BRAKE_PRESSURE_SENSE" (shape input) (at 135.89 81.28 180)
-    (effects (font (size 1.27 1.27)) (justify right))
-  )
-  (hierarchical_label "HITL_BRAKE_PRESSURE" (shape input) (at 55.88 50.8 180)
+  (label "BRAKE_PRESSURE_SENSE" (at 64.77 81.28 0)
+    (effects (font (size 1.27 1.27)) (justify left bottom))
+  )
+  (hierarchical_label "HITL_BRAKE_PRESSURE" (shape input) (at 55.88 48.26 180)
     (effects (font (size 1.27 1.27)) (justify right))
   )
@@
     (pin "P40")
   )
+  (symbol (lib_id "power:+5V") (at 58.42 76.2 0) (unit 1)
+    (in_bom yes) (on_board yes) (fields_autoplaced)
+    (property "Reference" "#PWR?" (id 0) (at 58.42 80.01 0)
+      (effects (font (size 1.27 1.27)) hide)
+    )
+    (property "Value" "+5V" (id 1) (at 58.42 71.12 0))
+    (property "Footprint" "" (id 2) (at 58.42 76.2 0)
+      (effects (font (size 1.27 1.27)) hide)
+    )
+    (property "Datasheet" "" (id 3) (at 58.42 76.2 0)
+      (effects (font (size 1.27 1.27)) hide)
+    )
+    (pin "1")
+  )
   (symbol (lib_id "formula:LED_0805") (at 201.93 105.41 90) (unit 1)
     (in_bom yes) (on_board yes)
@@
     (pin "2")
   )
+  (symbol (lib_id "power:GND") (at 58.42 86.36 0) (unit 1)
+    (in_bom yes) (on_board yes) (fields_autoplaced)
+    (property "Reference" "#PWR?" (id 0) (at 58.42 92.71 0)
+      (effects (font (size 1.27 1.27)) hide)
+    )
+    (property "Value" "GND" (id 1) (at 58.42 91.44 0))
+    (property "Footprint" "" (id 2) (at 58.42 86.36 0)
+      (effects (font (size 1.27 1.27)) hide)
+    )
+    (property "Datasheet" "" (id 3) (at 58.42 86.36 0)
+      (effects (font (size 1.27 1.27)) hide)
+    )
+    (pin "1")
+  )
   (symbol (lib_id "formula:TMUX1247DCKR") (at 66.04 49.53 0) (unit 1)
     (in_bom yes) (on_board yes) (fields_autoplaced)
@@
     (pin "1")
   )
-  (symbol (lib_id "Device:R_Potentiometer") (at 67.31 76.2 0) (unit 1)
+  (symbol (lib_id "Device:R_Potentiometer") (at 58.42 81.28 0) (unit 1)
     (in_bom yes) (on_board yes)
-    (property "Reference" "RV601" (id 0) (at 63.5 76.2 0))
-    (property "Value" "R_Potentiometer" (id 1) (at 67.31 66.04 0))
-    (property "Footprint" "footprints:PTV09A4020FB103" (id 2) (at 67.31 76.2 0)
-      (effects (font (size 1.27 1.27)) hide)
-    )
-    (property "Datasheet" "~" (id 3) (at 67.31 76.2 0)
-      (effects (font (size 1.27 1.27)) hide)
-    )
+    (property "Reference" "RV601" (id 0) (at 46.99 82.55 0))
+    (property "Value" "R_Potentiometer" (id 1) (at 46.99 80.01 0))
+    (property "Footprint" "footprints:PTV09A4020FB103" (id 2) (at 58.42 81.28 0)
+      (effects (font (size 1.27 1.27)) hide)
+    )
+    (property "Datasheet" "~" (id 3) (at 58.42 81.28 0)
+      (effects (font (size 1.27 1.27)) hide)
+    )
