File: vehicle/mkvi/hardware/rkh/air_control.kicad_sch (KiCad schematic)
At the start: 5 parts, among them J1101 Automotive_M.2

Commit message: switch micros and leds and adbms
Parts:
- D901, D902: symbol formula:LED_0805 -> OEM:LED_ORANGE
Changed lines of the file:
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@@
     (pin "2")
   )
-  (symbol (lib_id "formula:LED_0805") (at 209.55 104.14 90) (unit 1)
+  (symbol (lib_id "OEM:LED_ORANGE") (at 209.55 104.14 90) (unit 1)
     (in_bom yes) (on_board yes) (fields_autoplaced)
     (property "Reference" "D901" (id 0) (at 213.36 104.4701 90)
@@
     (pin "2")
   )
-  (symbol (lib_id "formula:LED_0805") (at 241.3 104.14 90) (unit 1)
+  (symbol (lib_id "OEM:LED_ORANGE") (at 241.3 104.14 90) (unit 1)
     (in_bom yes) (on_board yes) (fields_autoplaced)
     (property "Reference" "D902" (id 0) (at 245.11 104.4701 90)

Commit message: m.2 connectors
Parts:
- J1101: symbol formula:Automotive_M.2 -> OEM:Automotive_M.2
Changed lines of the file:
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@@
     (pin "1")
   )
-  (symbol (lib_id "formula:Automotive_M.2") (at 142.24 87.63 0) (unit 1)
+  (symbol (lib_id "OEM:Automotive_M.2") (at 142.24 87.63 0) (unit 1)
     (in_bom yes) (on_board yes) (fields_autoplaced)
     (property "Reference" "J1101" (id 0) (at 142.24 38.1 0)

Commit message: switch some resistors over
Parts:
- R902: symbol formula:R_10K -> OEM:10KR
- R903: symbol formula:R_1K -> OEM:1KR
Changed lines of the file:
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@@
     (pin "P40")
   )
-  (symbol (lib_id "formula:R_1K") (at 241.3 93.98 0) (unit 1)
+  (symbol (lib_id "OEM:1KR") (at 241.3 93.98 0) (unit 1)
     (in_bom yes) (on_board yes) (fields_autoplaced)
     (property "Reference" "R903" (id 0) (at 243.84 92.7099 0)
@@
     (pin "1")
   )
-  (symbol (lib_id "formula:R_10K") (at 209.55 93.98 0) (unit 1)
+  (symbol (lib_id "OEM:10KR") (at 209.55 93.98 0) (unit 1)
     (in_bom yes) (on_board yes) (fields_autoplaced)
     (property "Reference" "R902" (id 0) (at 212.09 92.7099 0)
