File: vehicle/mkvi/hardware/nostril/brakes/bspd.kicad_sch (KiCad schematic)
At the start: 33 parts, among them K1 G5Q-1A4-DC5-5V, Q2 SSM3K333R, Q3 SSM3K333R, SW1 SW_Push_SPST_NO, SW2 SW_Push_SPST_NO, U4 SN74LVC1G08DBVR, U5 MCP6001T-I-LT, U6 SN74LVC1G02DBVR, U7 SN74LVC1G02DBVR

Commit message: op amps
Parts:
- U5: symbol formula:MCP6001T-I-LT -> OEM:MCP6001
Changed lines of the file:
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@@
     (pin "2")
   )
-  (symbol (lib_id "formula:MCP6001T-I-LT") (at 139.7 60.96 0) (unit 1)
+  (symbol (lib_id "OEM:MCP6001") (at 139.7 60.96 0) (unit 1)
     (in_bom yes) (on_board yes)
     (property "Reference" "U5" (id 0) (at 140.97 64.77 0))

Commit message: swap logic gates and repair some files
Parts:
- U4: symbol formula:SN74LVC1G08DBVR -> OEM:SN74LVC1G08DBVR
- U6, U7: symbol formula:SN74LVC1G02DBVR -> OEM:SN74LVC1G02DBVR
Changed lines of the file:
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@@
     (pin "1")
   )
-  (symbol (lib_id "formula:SN74LVC1G02DBVR") (at 223.901 62.484 0) (unit 1)
+  (symbol (lib_id "OEM:SN74LVC1G02DBVR") (at 223.901 62.484 0) (unit 1)
     (in_bom yes) (on_board yes)
     (property "Reference" "U7" (id 0) (at 230.124 55.88 0)
@@
     (pin "1")
   )
-  (symbol (lib_id "formula:SN74LVC1G02DBVR") (at 186.69 62.611 0) (unit 1)
+  (symbol (lib_id "OEM:SN74LVC1G02DBVR") (at 186.69 62.611 0) (unit 1)
     (in_bom yes) (on_board yes)
     (property "Reference" "U6" (id 0) (at 192.913 56.007 0)
@@
     (pin "5")
   )
-  (symbol (lib_id "formula:SN74LVC1G08DBVR") (at 73.66 66.04 0) (unit 1)
+  (symbol (lib_id "OEM:SN74LVC1G08DBVR") (at 73.66 66.04 0) (unit 1)
     (in_bom yes) (on_board yes)
     (property "Reference" "U4" (id 0) (at 68.58 60.96 0)

Commit message: nmos
Parts:
- Q2, Q3: symbol formula:SSM3K333R -> OEM:SSM3K333R
Changed lines of the file:
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@@
     (pin "1")
   )
-  (symbol (lib_id "formula:SSM3K333R") (at 208.407 139.4968 0) (mirror y) (unit 1)
+  (symbol (lib_id "OEM:SSM3K333R") (at 208.407 139.4968 0) (mirror y) (unit 1)
     (in_bom yes) (on_board yes)
     (property "Reference" "Q2" (id 0) (at 208.153 135.1788 90)
@@
     (pin "1")
   )
-  (symbol (lib_id "formula:SSM3K333R") (at 211.4042 92.964 0) (unit 1)
+  (symbol (lib_id "OEM:SSM3K333R") (at 211.4042 92.964 0) (unit 1)
     (in_bom yes) (on_board yes)
     (property "Reference" "Q3" (id 0) (at 219.71 95.25 90)

Commit message: migrate ics and diodes
Parts:
- TP4, TP5, TP6: symbol formula:Test_Point_SMD -> OEM:TP_SMD
Changed lines of the file:
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@@
     (pin "1")
   )
-  (symbol (lib_id "formula:Test_Point_SMD") (at 83.82 64.77 0) (unit 1)
+  (symbol (lib_id "OEM:TP_SMD") (at 83.82 64.77 0) (unit 1)
     (in_bom yes) (on_board yes)
     (property "Reference" "TP4" (id 0) (at 82.55 57.15 0)
@@
     (pin "2")
   )
-  (symbol (lib_id "formula:Test_Point_SMD") (at 40.64 44.45 0) (unit 1)
+  (symbol (lib_id "OEM:TP_SMD") (at 40.64 44.45 0) (unit 1)
     (in_bom yes) (on_board yes)
     (property "Reference" "TP6" (id 0) (at 38.1 36.83 0)
@@
     (pin "1")
   )
-  (symbol (lib_id "formula:Test_Point_SMD") (at 219.964 138.2268 0) (mirror y) (unit 1)
+  (symbol (lib_id "OEM:TP_SMD") (at 219.964 138.2268 0) (mirror y) (unit 1)
     (in_bom yes) (on_board yes)
     (property "Reference" "TP5" (id 0) (at 217.424 134.4167 0)

Commit message: fuses, connectors, relays, misc
Parts:
- D2: value D_Zener_18V -> SMBJ5355B-TP; symbol formula:D_Zener_18V -> OEM:SMBJ5355B-TP
- K1: value G5Q-1A4-DC5-5V -> G5Q-1A4-DC5; symbol formula:G5Q-1A4-DC5-5V -> OEM:G5Q-1A4-DC5
- SW1, SW2: symbol formula:SW_Push_SPST_NO -> OEM:SW_Push_SPST_NO
Changed lines of the file:
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@@
     (pin "2")
   )
-  (symbol (lib_id "formula:D_Zener_18V") (at 188.341 144.9578 0) (unit 1)
+  (symbol (lib_id "OEM:SMBJ5355B-TP") (at 188.341 144.9578 0) (unit 1)
     (in_bom yes) (on_board yes)
     (property "Reference" "D2" (id 0) (at 187.96 149.86 0))
-    (property "Value" "D_Zener_18V" (id 1) (at 187.96 147.32 0))
+    (property "Value" "SMBJ5355B-TP" (id 1) (at 187.96 147.32 0))
     (property "Footprint" "footprints:DO-214AA" (id 2) (at 185.801 144.9578 0)
       (effects (font (size 1.27 1.27)) hide)
@@
     (pin "2")
   )
-  (symbol (lib_id "formula:SW_Push_SPST_NO") (at 26.67 50.8 0) (unit 1)
+  (symbol (lib_id "OEM:SW_Push_SPST_NO") (at 26.67 50.8 0) (unit 1)
     (in_bom yes) (on_board yes)
     (property "Reference" "SW2" (id 0) (at 26.67 46.99 0))
@@
     (pin "2")
   )
-  (symbol (lib_id "formula:SW_Push_SPST_NO") (at 26.67 76.2 0) (unit 1)
+  (symbol (lib_id "OEM:SW_Push_SPST_NO") (at 26.67 76.2 0) (unit 1)
     (in_bom yes) (on_board yes)
     (property "Reference" "SW1" (id 0) (at 26.67 72.39 0))
@@
     (pin "1")
   )
-  (symbol (lib_id "formula:G5Q-1A4-DC5-5V") (at 188.468 130.0988 90) (unit 1)
+  (symbol (lib_id "OEM:G5Q-1A4-DC5") (at 188.468 130.0988 90) (unit 1)
     (in_bom yes) (on_board yes)
     (property "Reference" "K1" (id 0) (at 188.468 119.3038 90))
-    (property "Value" "G5Q-1A4-DC5-5V" (id 1) (at 188.468 121.3358 90))
+    (property "Value" "G5Q-1A4-DC5" (id 1) (at 188.468 121.3358 90))
     (property "Footprint" "footprints:Relay_SPST_OMRON-G5Q-1A4_OEM" (id 2) (at 189.738 118.6688 0)
       (effects (font (size 1.27 1.27)) (justify left) hide)

Commit message: caps
Parts:
- C7: symbol formula:C_10uF -> OEM:10uF
- C9: symbol formula:C_1uF -> OEM:1uF
Changed lines of the file:
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@@
     (pin "1")
   )
-  (symbol (lib_id "formula:C_10uF") (at 107.95 63.5 180) (unit 1)
+  (symbol (lib_id "OEM:10uF") (at 107.95 63.5 180) (unit 1)
     (in_bom yes) (on_board yes)
     (property "Reference" "C7" (id 0) (at 101.6254 63.5762 0)
@@
     (pin "3")
   )
-  (symbol (lib_id "formula:C_1uF") (at 161.29 67.31 0) (unit 1)
+  (symbol (lib_id "OEM:1uF") (at 161.29 67.31 0) (unit 1)
     (in_bom yes) (on_board yes) (fields_autoplaced)
     (property "Reference" "C9" (id 0) (at 165.1 64.7699 0)

Commit message: resistors
Parts:
- C10, C11, C12, C6, C8: symbol OEM:0.1uF -> OEM:0u1F
- R10, R17: symbol formula:R_200 -> OEM:200R
- R11: symbol formula:R_71.5k -> OEM:71K5R
Changed lines of the file:
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@@
     (pin "2")
   )
-  (symbol (lib_id "OEM:0.1uF") (at 66.294 51.7906 90) (unit 1)
+  (symbol (lib_id "OEM:0u1F") (at 66.294 51.7906 90) (unit 1)
     (in_bom yes) (on_board yes)
     (property "Reference" "C6" (id 0) (at 67.564 44.1706 90)
@@
     (pin "2")
   )
-  (symbol (lib_id "OEM:0.1uF") (at 194.31 48.641 270) (unit 1)
+  (symbol (lib_id "OEM:0u1F") (at 194.31 48.641 270) (unit 1)
     (in_bom yes) (on_board yes)
     (property "Reference" "C10" (id 0) (at 193.04 44.831 90)
@@
     (pin "1")
   )
-  (symbol (lib_id "formula:R_200") (at 245.0084 69.088 0) (unit 1)
+  (symbol (lib_id "OEM:200R") (at 245.0084 69.088 0) (unit 1)
     (in_bom yes) (on_board yes)
     (property "Reference" "R17" (id 0) (at 242.9764 69.977 90)
@@
     (pin "1")
   )
-  (symbol (lib_id "OEM:0.1uF") (at 195.3006 98.8314 180) (unit 1)
+  (symbol (lib_id "OEM:0u1F") (at 195.3006 98.8314 180) (unit 1)
     (in_bom yes) (on_board yes)
     (property "Reference" "C11" (id 0) (at 200.3806 98.7044 90))
@@
     (pin "1")
   )
-  (symbol (lib_id "formula:R_200") (at 83.82 82.55 180) (unit 1)
+  (symbol (lib_id "OEM:200R") (at 83.82 82.55 180) (unit 1)
     (in_bom yes) (on_board yes) (fields_autoplaced)
     (property "Reference" "R10" (id 0) (at 81.28 83.8201 0)
@@
     (pin "5")
   )
-  (symbol (lib_id "formula:R_71.5k") (at 100.33 58.42 90) (unit 1)
+  (symbol (lib_id "OEM:71K5R") (at 100.33 58.42 90) (unit 1)
     (in_bom yes) (on_board yes) (fields_autoplaced)
     (property "Reference" "R11" (id 0) (at 100.33 52.07 90))
@@
     (pin "1")
   )
-  (symbol (lib_id "OEM:0.1uF") (at 144.78 48.26 270) (unit 1)
+  (symbol (lib_id "OEM:0u1F") (at 144.78 48.26 270) (unit 1)
     (in_bom yes) (on_board yes)
     (property "Reference" "C8" (id 0) (at 143.51 44.45 90)
@@
     (pin "2")
   )
-  (symbol (lib_id "OEM:0.1uF") (at 231.521 48.514 270) (unit 1)
+  (symbol (lib_id "OEM:0u1F") (at 231.521 48.514 270) (unit 1)
     (in_bom yes) (on_board yes)
     (property "Reference" "C12" (id 0) (at 230.251 44.704 90)
