File: vehicle/mkvi/hardware/nostril/motherboard/nostril.kicad_pcb (KiCad board)
At the start: 2 copper layers, 314.3 x 82.6 mm, 40 parts, among them J1 Ampseal_23_RA, J2 Ampseal_23_RA, J3 Ampseal_23_RA, J4 Automotive_M.2, J5 Automotive_M.2, J6 Automotive_M.2, J7 Automotive_M.2, J8 MicroFit_RA_4, U1 MP1477HGTF-P

Commit message: update silkscreen and add CAN term
Parts:
- removed kibuzzard-63FE2473: G***, kibuzzard-63FE2473
- removed kibuzzard-63FE2479: G***, kibuzzard-63FE2479
- removed kibuzzard-63FE24B0: G***, kibuzzard-63FE24B0
- removed kibuzzard-63FE24BA: G***, kibuzzard-63FE24BA
- added G***: LOGO, LOGO, B.Cu at (22.2, 93.6)
- added G***: LOGO, footprints:OE_Logo_ft, B.Cu at (141.5, 83.7)
- added R9: R_120_DNP, footprints:R_0805_OEM, F.Cu at (-15.0, 70.8)
- added REF**: OEM_Logo_15_mm, OEM:OEM_Logo_15_mm, F.Cu at (-23.1, 123.4)
- added kibuzzard-63FE478D: G***, kibuzzard-63FE478D, F.Cu at (72.1, 69.1)
- added kibuzzard-63FE479B: G***, kibuzzard-63FE479B, F.Cu at (72.3, 101.1)
- added kibuzzard-63FE47A2: G***, kibuzzard-63FE47A2, F.Cu at (171.4, 80.0)
- added kibuzzard-63FE47AC: G***, kibuzzard-63FE47AC, F.Cu at (228.9, 90.7)
- added kibuzzard-63FE4A40: G***, kibuzzard-63FE4A40, F.Cu at (15.4, 120.6)
Routing:
- net /CAN_+: track 426.4 -> 426.9 mm
Other:
- board text added: "Amit Kumar-Hermosillo R1 2.28.23"

Commit message: final touches
Parts:
- added QR*****: https://coda.io/d/Documentation_dbuFnC2EA_e/Low-Voltage-Sys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, https:__coda.io_d_Documentation_dbuFnC2EA_e_Low-Voltage-Syste, B.Cu at (224.2, 86.8)
- added kibuzzard-63FE5D89: G***, kibuzzard-63FE5D89, B.Cu at (224.6, 99.1)
- added kibuzzard-63FE5E2A: G***, kibuzzard-63FE5E2A, F.Cu at (224.9, 53.5)
- added kibuzzard-63FE5E61: G***, kibuzzard-63FE5E61, F.Cu at (140.9, 111.8)
- added kibuzzard-63FE5E77: G***, kibuzzard-63FE5E77, F.Cu at (206.0, 111.5)

Commit message: Commit Rev 2; Respond to PR feedback
Parts:
- added ?: , , F.Cu at (261.5, 123.1)
- added ?: , , F.Cu at (-35.1, 123.1)
- added ?: , , F.Cu at (261.5, 58.3)
- added REF**: Mounting_Hole_4-40, footprints:Mounting_Hole_4-40, F.Cu at (-35.1, 58.3)
- added REFe: MountingHole_440_Keystone_4939, OEM:MountingHole_440_Keystone_4939, F.Cu at (93.0, 76.7)
- added REFe: MountingHole_440_Keystone_4939, OEM:MountingHole_440_Keystone_4939, F.Cu at (12.9, 69.3)
- added REFe: MountingHole_440_Keystone_4939, OEM:MountingHole_440_Keystone_4939, F.Cu at (196.7, 91.4)
- added REFe: MountingHole_440_Keystone_4939, OEM:MountingHole_440_Keystone_4939, F.Cu at (-5.52, 101.4)
- added kibuzzard-63FF646A: G***, kibuzzard-63FF646A, F.Cu at (-19.6, 61.2)
- J1, J2, J3: footprint footprints:Ampseal_23 -> OEM:Ampseal_23_RA
- J8: value MicroFit_RA_4 -> MicroFit_VT_4; footprint footprints:MicroFit_RA_4 -> footprints:MicroFit_VT_4
- QR*****, kibuzzard-63FE5D89: moved to F.Cu
- moved kibuzzard-63FE5D89 126.2 mm to (101.1, 124.7), turned to 0 degrees
- moved QR***** 125.4 mm to (101.5, 112.5), turned to 0 degrees
- moved J3 41.0 mm to (244.8, 58.8), turned to 180 degrees
- moved L1 23.0 mm to (260.2, 110.6)
- moved F2 22.5 mm to (259.8, 100.3), turned to 90 degrees
- moved C5 19.2 mm to (254.9, 102.3), turned to 180 degrees
- moved C6 19.1 mm to (254.9, 104.7), turned to 180 degrees
- moved C3 17.4 mm to (249.2, 111.1), turned to 0 degrees
- moved F1 15.7 mm to (235.1, 124.8), turned to 0 degrees
- moved kibuzzard-63FE5E2A 14.2 mm to (224.9, 67.8)
- moved R3 13.5 mm to (249.2, 113.2)
- moved U1 9.61 mm to (254.4, 118.0), turned to 180 degrees
- moved C1 9.43 mm to (254.3, 123.5), turned to 180 degrees
- moved C2 8.04 mm to (254.2, 120.3), turned to 180 degrees
- moved C4 7.77 mm to (245.8, 120.7)
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Routing:
- net /SHDN_BOTS_IN: track 152.7 -> 204.1 mm
- net /SHDN_BOTS_OUT: track 233.9 -> 269.5 mm, vias 4 -> 2
- net /SUS_TRAVEL_R_SIG: track 34.6 -> 64.4 mm
- net +BATT: track 171.1 -> 144.4 mm
- net /SUS_TRAVEL_L_SIG: track 36.9 -> 59.1 mm
- net Net-(C1-Pad1): track 391.3 -> 407.0 mm, vias 2 -> 3
- net /INPUT_THROTTLE_1: track 133.6 -> 147.7 mm
- net /BRAKE_PRESSURE_SENSE: track 155.2 -> 168.7 mm
- net /WHEEL_SPEED_R_SIG: track 39.4 -> 52.1 mm, vias 0 -> 2
- net Net-(R4-Pad1): track 13.1 -> 2.87 mm
- net Net-(C4-Pad2): track 15.4 -> 23.1 mm, vias 0 -> 2
- net /INPUT_THROTTLE_2: track 135.0 -> 142.7 mm
- net GND: track 72.8 -> 66.0 mm, vias 39 -> 103
- net +5V: track 0.00 -> 6.11 mm, vias 0 -> 6
- net /WHEEL_SPEED_L_SIG: track 42.4 -> 48.0 mm, vias 0 -> 2
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- added copper zone on F.Cu, net GND
- added copper zone on F.Cu, net Net-(C3-Pad2)
- added copper zone on F.Cu, net Net-(C4-Pad2)
Other:
- outline, holes or cut-outs redrawn

Commit message: fix nostril dimensions
Parts:
- moved kibuzzard-63FE5E2A 7.87 mm to (224.3, 59.9)
- moved J3 7.85 mm to (244.9, 50.9)
Routing:
- net Net-(C1-Pad1): track 407.0 -> 416.6 mm
- net /SUS_TRAVEL_R_SIG: track 64.4 -> 72.5 mm
- net /SUS_TRAVEL_L_SIG: track 59.1 -> 67.2 mm
- net /INPUT_THROTTLE_1: track 147.7 -> 155.6 mm
- net /INPUT_THROTTLE_2: track 142.7 -> 149.2 mm, vias 2 -> 4
- net /WHEEL_SPEED_L_SIG: track 48.0 -> 53.9 mm
- net /WHEEL_SPEED_R_SIG: track 52.1 -> 57.5 mm
- net /BRAKE_PRESSURE_SENSE: track 168.7 -> 173.3 mm
- net /SHDN_BOTS_OUT: track 269.5 -> 272.6 mm
- net /SHDN_BOTS_IN: track 204.1 -> 206.9 mm
- net +5V: track 6.11 -> 6.68 mm
Other:
- board size 314.3 x 82.6 mm -> 314.4 x 90.3 mm

Commit message: r2
Parts:
- added JP1: SolderJumper_2_Open, Jumper:SolderJumper-2_P1.3mm_Open_RoundedPad1.0x1.5mm, F.Cu at (-12.7, 66.7)
- moved F1 4.67 mm to (238.8, 121.9)
- moved REF** 3.68 mm to (-35.1, 54.6)
Connections:
- J3 pad 3: +5V -> /THROTTLE_1+
- J3 pad 4: +5V -> /THROTTLE_2+
- J5 pad 13: +5V -> /THROTTLE_1+
- J5 pad 15: +5V -> /THROTTLE_2+
- R9 pad 2: /CAN_- -> Net-(JP1-A)
Routing:
- net /THROTTLE_1+: track 0.00 -> 149.4 mm, vias 0 -> 2
- net /THROTTLE_2+: track 0.00 -> 147.3 mm, vias 0 -> 2
- net +BATT: track 144.4 -> 149.3 mm
- net Net-(U1-VIN): track 416.6 -> 411.7 mm
- net Net-(JP1-A): track 0.00 -> 2.50 mm
- net /CAN_-: track 415.7 -> 417.0 mm
Other:
- board text added: "Amit Kumar-Hermosillo R2 9.9.23"
- board text removed: "Amit Kumar-Hermosillo R1 2.28.23"
