File: tutorials/eLeads/darian/analog.kicad_sch (KiCad schematic)
At the start: 22 parts, among them SW1 SW_SPDT, SW2 SW_SPDT, U6 ${SIM.PARAMS}, U7 ${SIM.PARAMS}, U8 ${SIM.PARAMS}

Commit message: Create initial PCB
Parts:
- U6: footprint Capacitor_SMD:C_0402_1005Metric -> Package_TO_SOT_THT:Heraeus_TO-92-2
- U7, U8: footprint Capacitor_SMD:C_0805_2012Metric -> Package_TO_SOT_THT:Heraeus_TO-92-2
Changed lines of the file:
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@@
       (effects (font (size 1.27 1.27)))
     )
-    (property "Footprint" "Capacitor_SMD:C_0805_2012Metric" (at 82.55 76.2 0)
+    (property "Footprint" "Package_TO_SOT_THT:Heraeus_TO-92-2" (at 82.55 76.2 0)
       (effects (font (size 1.27 1.27)) hide)
     )
@@
       (effects (font (size 1.27 1.27)))
     )
-    (property "Footprint" "Capacitor_SMD:C_0402_1005Metric" (at 82.55 43.18 0)
+    (property "Footprint" "Package_TO_SOT_THT:Heraeus_TO-92-2" (at 82.55 43.18 0)
       (effects (font (size 1.27 1.27)) hide)
     )
@@
       (effects (font (size 1.27 1.27)))
     )
-    (property "Footprint" "Capacitor_SMD:C_0805_2012Metric" (at 129.54 59.69 0)
-      (effects (font (size 1.27 1.27)) hide)
-    )
+    (property "Footprint" "Package_TO_SOT_THT:Heraeus_TO-92-2" (at 129.54 59.69 0)
+      (effects (font (size 1.27 1.27)) hide)
+    )

Commit message: Revise PCB
Parts:
- U6, U7, U8: footprint Package_TO_SOT_THT:Heraeus_TO-92-2 -> Package_TO_SOT_SMD:VSOF5
Connections:
- net SIGNAL_A renamed ANALOG_A
- net SIGNAL_B renamed ANALOG_B
Changed lines of the file:
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@@
     (effects (font (size 2 2)) (justify left bottom))
   )
-  (label "SIGNAL_B" (at 50.8 64.77 0) (fields_autoplaced)
+  (label "ANALOG_B" (at 50.8 64.77 0) (fields_autoplaced)
     (effects (font (size 1.27 1.27)) (justify left bottom))
   )
-  (label "SIGNAL_A" (at 50.8 31.75 0) (fields_autoplaced)
+  (label "ANALOG_A" (at 50.8 31.75 0) (fields_autoplaced)
     (effects (font (size 1.27 1.27)) (justify left bottom))
   )
@@
       (effects (font (size 1.27 1.27)))
     )
-    (property "Footprint" "Package_TO_SOT_THT:Heraeus_TO-92-2" (at 82.55 76.2 0)
+    (property "Footprint" "Package_TO_SOT_SMD:VSOF5" (at 82.55 76.2 0)
       (effects (font (size 1.27 1.27)) hide)
     )
@@
       (effects (font (size 1.27 1.27)))
     )
-    (property "Footprint" "Package_TO_SOT_THT:Heraeus_TO-92-2" (at 82.55 43.18 0)
+    (property "Footprint" "Package_TO_SOT_SMD:VSOF5" (at 82.55 43.18 0)
       (effects (font (size 1.27 1.27)) hide)
     )
@@
       (effects (font (size 1.27 1.27)))
     )
-    (property "Footprint" "Package_TO_SOT_THT:Heraeus_TO-92-2" (at 129.54 59.69 0)
-      (effects (font (size 1.27 1.27)) hide)
-    )
+    (property "Footprint" "Package_TO_SOT_SMD:VSOF5" (at 129.54 59.69 0)
+      (effects (font (size 1.27 1.27)) hide)
+    )
