File: tutorials/eLeads/darian/darian.kicad_pcb (KiCad board)
At the start: 2 copper layers, 65 parts, among them J2 MicroFit_RA_4, J3 MicroFit_RA_4, Q1 BC547, Q2 SSM3K333R, Q3 SSM3K333R, SW1 SW_SPDT, SW2 SW_SPDT, U1 TC1262-33, U2 ATMEGA16M1, U3 BMP280, U4 RFM69HCW, U5 TJA1042T, U6 ${SIM.PARAMS}, U7 ${SIM.PARAMS}, U8 ${SIM.PARAMS}, Y1 Crystal_12MHz

Commit message: Create initial PCB
Parts:
- added J1: CONN_02X03, Connector_Harwin:Harwin_LTek-Male_2x03_P2.00mm_Vertical, F.Cu at (164.9, 63.0)
- added K1: G5Q-1A4-DC5-5V, Relay_THT:Relay_SPST_Omron-G5Q-1A, F.Cu at (89.5, 123.2)
- added K2: G5Q-1A4-DC5-5V, Relay_THT:Relay_SPST_Omron-G5Q-1A, F.Cu at (116.8, 115.6)
- J2, J3: footprint Connector_Molex:Molex_KK-396_A-41791-0004_1x04_P3.96mm_Vertical -> Connector_Molex:Molex_Micro-Fit_3.0_43045-0412_2x02_P3.00mm_Vertical
- U6: footprint Capacitor_SMD:C_0402_1005Metric -> Package_TO_SOT_SMD:VSOF5
- U7, U8: footprint Capacitor_SMD:C_0805_2012Metric -> Package_TO_SOT_SMD:VSOF5
- moved C10 79.1 mm to (76.8, 60.3), turned to 180 degrees
- moved C11 78.9 mm to (76.7, 62.9), turned to 180 degrees
- moved RV1 73.0 mm to (114.8, 131.4)
- moved U1 72.7 mm to (122.0, 60.3), turned to -90 degrees
- moved C12 72.5 mm to (150.2, 66.7)
- moved RV2 70.8 mm to (114.8, 141.6)
- moved C3 69.9 mm to (113.8, 57.1)
- moved C7 69.7 mm to (139.4, 57.3)
- moved C8 69.7 mm to (139.4, 60.3)
- moved C4 67.3 mm to (128.7, 57.1)
- moved Q2 61.3 mm to (88.0, 128.3)
- moved R15 59.1 mm to (108.8, 141.6), turned to 180 degrees
- moved R4 56.8 mm to (134.0, 64.9)
- moved R5 55.3 mm to (134.0, 69.4)
- moved R6 55.3 mm to (134.0, 57.3)
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Routing:
- net GND: track 0.00 -> 164.9 mm, vias 0 -> 10
- net SHDN_IN: track 0.00 -> 53.3 mm, vias 0 -> 2
- net SHDN_OUT: track 0.00 -> 40.3 mm, vias 0 -> 2
- net +5V: track 0.00 -> 39.2 mm
- net Net-(U2-AVCC): track 0.00 -> 32.8 mm, vias 0 -> 4
- net Net-(R18-Pad2): track 0.00 -> 15.0 mm
- net Net-(R20-Pad2): track 0.00 -> 14.8 mm
- net Net-(U2-(PCINT25/OC0B/XTAL1)PE1): track 0.00 -> 14.7 mm
- net Net-(U6--): track 0.00 -> 13.4 mm
- net Net-(U7--): track 0.00 -> 13.4 mm
- net Net-(U2-(PCINT26/ADC0/XTAL2)PE2): track 0.00 -> 13.1 mm
- net Net-(U1-VI): track 0.00 -> 12.6 mm
- net Net-(Q1-B): track 0.00 -> 12.1 mm, vias 0 -> 2
- net +3.3V: track 0.00 -> 11.6 mm
- net Net-(SW1-C): track 0.00 -> 11.2 mm
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
Commit message: Revise PCB
Parts:
- moved C5 26.9 mm to (112.8, 84.0)
- moved C6 26.9 mm to (107.7, 84.0)
- moved C1 26.9 mm to (104.0, 72.9)
- moved C2 26.9 mm to (104.0, 67.9)
- moved R1 26.9 mm to (104.0, 78.0)
- moved U2 26.9 mm to (112.1, 73.5)
- moved Y1 26.9 mm to (110.2, 88.7)
- moved R8 18.5 mm to (109.3, 66.5), turned to 0 degrees
- moved TP1 10.8 mm to (168.3, 102.9)
- moved TP4 9.19 mm to (168.3, 117.2)
- moved R3 3.95 mm to (113.7, 63.4)
- moved C12 2.63 mm to (149.5, 64.1)
- moved J1 2.63 mm to (164.3, 60.4)
- moved U5 2.63 mm to (151.8, 59.1)
- moved R13 2.63 mm to (154.3, 64.1)
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Connections:
- net /Analog Section/SIGNAL_A renamed /Analog Section/ANALOG_A
- net /Analog Section/SIGNAL_B renamed /Analog Section/ANALOG_B
- net SHDN_IN renamed /SHDN_IN
- net SHDN_OUT renamed /SHDN_OUT
Routing:
- net /ANALOG_A: track 0.00 -> 97.7 mm, vias 0 -> 2
- net /SENSOR_SS: track 0.00 -> 96.2 mm, vias 0 -> 2
- net /ANALOG_B: track 0.00 -> 89.2 mm, vias 0 -> 2
- net /ANALOG_SS: track 0.00 -> 88.5 mm
- net /SCK: track 3.73 -> 91.3 mm, vias 0 -> 5
- net Net-(TP1-TP): track 0.00 -> 71.5 mm
- net GND: track 164.9 -> 118.4 mm, vias 10 -> 23
- net /MOSI: track 6.71 -> 45.5 mm
- net +5V: track 39.2 -> 75.6 mm, vias 0 -> 5
- net /MISO: track 0.00 -> 33.3 mm, vias 0 -> 3
- net Net-(U8-+): track 10.7 -> 42.5 mm
- net /NSS: track 0.00 -> 31.0 mm, vias 0 -> 2
- net /Analog Section/ANALOG_OUT: track 0.00 -> 28.1 mm
- net Net-(U8--): track 10.2 -> 38.1 mm
- net Net-(U3-VDD): track 0.00 -> 7.71 mm, vias 0 -> 2
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
Commit message: Revise PCB again
Parts:
- moved R13 5.63 mm to (157.0, 59.2), turned to -90 degrees
Routing:
- net +5V: track 75.6 -> 250.4 mm, vias 5 -> 8
- net /ANALOG_SS: track 88.5 -> 135.3 mm
- net Net-(U5-CANL): track 0.00 -> 2.83 mm
- net Net-(U5-CANH): track 0.00 -> 2.73 mm
Other:
- board text added: "Analog Section"
- board text added: "Can Transceiver"
- board text added: "Pressure Sensor"
- board text added: "Programming Header"
- board text added: "RF Module"
- board text added: "Shutdown Node"
