File: projects/stm32g431_dev_board/stm32g431_dev_board.kicad_pcb (KiCad board)
At the start: 2 copper layers, 30 parts, among them J1 Barrel_jack, J10 CONN_01X03, J12 Screw_Terminal_01x03, J14 CONN_01x02, SW1 SW_Push_SPST_NO, SW2 SW_Push_SPST_NO, SW3 SW_Push_SPST_NO, U1 AP7370, U2 STM32F103C8Tx, Y1 Crystal_SMD

Commit message: finish sch
Parts:
- removed C10, C3, C7, C8, C9: C_100nF, footprints:C_0603_1608Metric
- removed C6: C_1uF, footprints:C_0805_OEM
- removed D3: LED_0805, footprints:LED_0805_OEM
- removed D4: LED_0805_Amber, footprints:LED_0805_OEM
- removed J1: Barrel_jack, footprints:barrel_jack_PJ-037A
- removed J10: CONN_01X03, footprints:PinHeader_1x03_P2.54mm_Vertical
- removed J12: Screw_Terminal_01x03, TerminalBlock_Phoenix:TerminalBlock_Phoenix_MKDS-1,5-3_1x03_P5.00mm_Horizontal
- removed J14: CONN_01x02, Connector_PinSocket_2.54mm:PinSocket_1x02_P2.54mm_Vertical
- removed SW2, SW3: SW_Push_SPST_NO, footprints:SW_B3U-1000P_4.2x1.7mm
- removed TP1, TP2, TP3: Test_Point_SMD, footprints:Test_Point_SMD
- removed U1: AP7370, footprints:SOT-23-5
- removed U2: STM32F103C8Tx, Package_QFP:LQFP-48_7x7mm_P0.5mm
- removed Y1: Crystal_SMD, footprints:Crystal_SMD_FA238
- added C12: C_4.7uF, footprints:C_0603_1608Metric, F.Cu at (128.8, 103.3)
- added C13: C_100pF, footprints:C_0603_1608Metric, F.Cu at (128.8, 105.8)
- added C14: C_100pF, footprints:C_0603_1608Metric, F.Cu at (128.8, 108.3)
- added C15: C_1uF, footprints:C_0603_1608Metric, F.Cu at (132.8, 95.8)
- added C16: C_100nF, footprints:C_0603_1608Metric, F.Cu at (132.8, 98.3)
- added C17: C_100nF, footprints:C_0603_1608Metric, F.Cu at (132.8, 100.8)
- added C18: C_100nF, footprints:C_0603_1608Metric, F.Cu at (132.8, 103.3)
- added C19: C_100nF, footprints:C_0603_1608Metric, F.Cu at (132.8, 105.8)
- added C20: C_10uF, footprints:C_0603_1608Metric, F.Cu at (132.8, 108.3)
- added C21: C_100nF, footprints:C_0603_1608Metric, F.Cu at (136.8, 95.8)
- added D10: EAST16084WA1, footprints:WL-SMCD_0603, F.Cu at (161.0, 108.5)
- added D11: EAST16084WA1, footprints:WL-SMCD_0603, F.Cu at (161.0, 110.7)
- added D5: USBLC6-2SC6, footprints:SOT-23-6_OEM, F.Cu at (148.5, 81.8)
- added D6: SMAJ24A, footprints:SMAJ24A-13-F, F.Cu at (158.2, 103.0)
- added D7: NUP2105LT1G, footprints:SOT-23-3_OEM, F.Cu at (147.5, 86.4)
- added D8: ESDALC6V1W5, footprints:SOT323-5L, F.Cu at (149.8, 107.8)
- added D9: ESDALC6V1W5, footprints:SOT323-5L, F.Cu at (152.5, 107.8)
- added F1: MF-NSMF025_30X-2, footprints:MFNSMF02530X2, F.Cu at (154.5, 86.0)
- added F2: MF-NSMF025_30X-2, footprints:MFNSMF02530X2, F.Cu at (154.5, 90.7)
- added FL1: ACM2012, footprints:ACM2012-201-2P-T002.kicad_mod, F.Cu at (150.8, 111.1)
- added IC1: STM32G431CBT6, footprints:QFP50P900X900X160-48N, F.Cu at (148.5, 100.2)
- added J5: 2601-1104, footprints:26011104, F.Cu at (131.5, 80.5)
- added J6: 2171790001, footprints:MOLEX_2171790001, F.Cu at (156.6, 79.6)
- added R10: R_60.4, footprints:R_0603_1608Metric, F.Cu at (140.8, 98.3)
- added R11: R_60.4, footprints:R_0603_1608Metric, F.Cu at (140.8, 100.8)
- added R12: R_47, footprints:R_0603_1608Metric, F.Cu at (140.8, 103.3)
- added R13: R_1k, footprints:R_0603_1608Metric, F.Cu at (140.8, 105.8)
- added R14: R_1k, footprints:R_0603_1608Metric, F.Cu at (140.8, 108.3)
- added R4: R_10k, footprints:R_0603_1608Metric, F.Cu at (136.8, 103.3)
- added R9: R_22, footprints:R_0603_1608Metric, F.Cu at (140.8, 95.8)
- added SW4: GW12LBP, footprints:GW12LBP, F.Cu at (156.6, 108.8)
- added SW5: SW_NO, footprints:SW_B3U-1000P_4.2x1.7mm, F.Cu at (143.9, 110.5)
- added U3: AP7375-33SA-7, footprints:SOT-23-3_OEM, F.Cu at (147.5, 91.1)
- added U8: TCAN3413DR, footprints:SOIC-8_3.9x4.9mm_Pitch1.27mm_OEM, F.Cu at (158.4, 97.7)
- added Y2: 32KHz, footprints:Crystal_SMD_FA238, F.Cu at (160.6, 85.8)
- added Y3: 24MHz, footprints:Crystal_SMD_FA238, F.Cu at (160.6, 89.9)
- C11: value C_0.1uF -> C_1uF; footprint footprints:C_0805_OEM -> footprints:C_0603_1608Metric
- C4: footprint footprints:C_0805_OEM -> footprints:C_0603_1608Metric
- C5: value C_1uF -> C_0.1uF; footprint footprints:C_0805_OEM -> footprints:C_0603_1608Metric
- D1: value LED_0805 -> EAST16084WA1; footprint footprints:LED_0805_OEM -> footprints:WL-SMCD_0603
- D2: value LED_0805 -> PMEG3005CT,215; footprint footprints:LED_0805_OEM -> footprints:SOT-23-3_OEM
- R2: value R_1K -> R_5.1k; footprint footprints:R_0805_OEM -> footprints:R_0603_1608Metric
- R3: value R_200 -> R_5.1k; footprint footprints:R_0805_OEM -> footprints:R_0603_1608Metric
- R5: value R_0_2512 -> R_1k; footprint footprints:R_2512_OEM -> footprints:R_0603_1608Metric
- R8: value R_120 -> R_22; footprint footprints:R_0805_OEM -> footprints:R_0603_1608Metric
- SW1: value SW_Push_SPST_NO -> SW_NO
- moved D2 93.2 mm to (147.5, 77.1)
- moved R5 81.2 mm to (136.8, 105.8)
- moved D1 80.3 mm to (161.0, 106.2)
- moved C11 74.2 mm to (128.8, 100.8)
- moved C5 71.3 mm to (128.8, 98.3)
- moved C4 71.0 mm to (128.8, 95.8)
- moved SW1 63.4 mm to (143.9, 107.4)
- moved R3 62.1 mm to (136.8, 100.8)
- moved R2 61.8 mm to (136.8, 98.3)
- moved R8 58.2 mm to (136.8, 108.3)
Connections:
- C11 pad 1: +3.3V -> Net-(U3-Vin)
- C4 pad 1: +12V -> +3V3
- C5 pad 1: Net-(U1-Vout) -> +3V3
- D1 pad 2: Net-(D1-A) -> Net-(D1-Pad2)
- D2 pad 1: GND -> +VIN
- D2 pad 2: Net-(D2-A) -> +VUSB
- R2 pad 1: +12V -> Net-(J6-CC2)
- R2 pad 2: Net-(D1-A) -> GND
- R3 pad 1: Net-(U1-Vout) -> Net-(J6-CC1)
- R3 pad 2: Net-(D2-A) -> GND
- R5 pad 1: +5V -> +3V3
- R5 pad 2: Net-(U1-Vout) -> Net-(D1-Pad2)
- R8 pad 2: /CAN1_- -> /USB_DN
- SW1 pad 1: /NRST -> /nRESET

Commit message: begin layout
Parts:
- removed C18, C19, C21: C_100nF, footprints:C_0603_1608Metric
- removed C20: C_10uF, footprints:C_0603_1608Metric
- removed D11: EAST16084WA1, footprints:WL-SMCD_0603
- removed R13, R14: R_1k, footprints:R_0603_1608Metric
- removed SW4: GW12LBP, footprints:GW12LBP
- removed SW5: SW_NO, footprints:SW_B3U-1000P_4.2x1.7mm
- removed U3: AP7375-33SA-7, footprints:SOT-23-3_OEM
- removed U8: TCAN3413DR, footprints:SOIC-8_3.9x4.9mm_Pitch1.27mm_OEM
- removed Y3: 24MHz, footprints:Crystal_SMD_FA238
- added C1: C_6.8uF, footprints:C_0603_1608Metric, F.Cu at (168.6, 102.5)
- added C10: C_10uF, footprints:C_0603_1608Metric, F.Cu at (248.4, 132.6)
- added C2: C_6.8uF, footprints:C_0603_1608Metric, F.Cu at (168.6, 105.0)
- added C3: C_5.1uF, footprints:C_0603_1608Metric, F.Cu at (168.6, 107.5)
- added C6: C_100nF, footprints:C_0603_1608Metric, F.Cu at (168.6, 115.0)
- added C7: C_100nF, footprints:C_0603_1608Metric, F.Cu at (168.6, 117.5)
- added C8: C_100nF, footprints:C_0603_1608Metric, F.Cu at (168.6, 120.0)
- added C9: C_1uF, footprints:C_0603_1608Metric, F.Cu at (246.6, 123.7)
- added D3: EAST16084WA1, footprints:WL-SMCD_0603, F.Cu at (170.6, 90.0)
- added D4: EAST16084WA1, footprints:WL-SMCD_0603, F.Cu at (170.6, 92.2)
- added J1: 2171790001, footprints:MOLEX_2171790001, F.Cu at (197.4, 95.0)
- added J2: 2601-1104, footprints:26011104, F.Cu at (270.8, 98.9)
- added J3: MicroFit_V_2, footprints:MicroFit_V_2, F.Cu at (196.1, 69.5)
- added J4: Samtec FTSH, footprints:SAMTEC_FTSH-105-01-LM-D-K, F.Cu at (244.2, 71.7)
- added J7: Conn_01x03, Connector_PinHeader_2.54mm:PinHeader_1x03_P2.54mm_Vertical, F.Cu at (239.9, 62.5)
- added JP1: Jumper, footprints:SolderJumper-2_Open_Hooks0.8x1.8mm, F.Cu at (255.5, 94.6)
- added JP2: Jumper, footprints:SolderJumper-2_Open_Hooks0.8x1.8mm, F.Cu at (255.5, 97.4)
- added R1: R_1k, footprints:R_0603_1608Metric, F.Cu at (234.7, 114.8)
- added R6: R_1k, footprints:R_0603_1608Metric, F.Cu at (170.1, 85.5)
- added R7: R_200, footprints:R_0603_1608Metric, F.Cu at (238.2, 119.1)
- added SW2: SW_NO, footprints:SW_B3U-1000P_4.2x1.7mm, F.Cu at (187.5, 121.1)
- added SW3: GW12LBP, footprints:GW12LBP, F.Cu at (259.5, 90.2)
- added TP1: TestPoint_Probe, footprints:TestPoint_Hole_D1mm, F.Cu at (172.4, 133.7)
- added TP10: TestPoint_Probe, footprints:TestPoint_Hole_D1mm, F.Cu at (178.4, 133.7)
- added TP11: TestPoint_Probe, footprints:TestPoint_Hole_D1mm, F.Cu at (178.4, 135.7)
- added TP12: TestPoint_Probe, footprints:TestPoint_Hole_D1mm, F.Cu at (178.4, 137.7)
- added TP13: TestPoint_Probe, footprints:TestPoint_Hole_D1mm, F.Cu at (180.4, 133.7)
- added TP14: CANH, TestPoint:TestPoint_Keystone_5000-5004_Miniature, F.Cu at (251.8, 91.3)
- added TP15: CANL, TestPoint:TestPoint_Keystone_5000-5004_Miniature, F.Cu at (248.4, 91.3)
- added TP16: TestPoint_Probe, footprints:TestPoint_Hole_D1mm, F.Cu at (206.4, 95.0)
- added TP17: CANH, TestPoint:TestPoint_Keystone_5000-5004_Miniature, F.Cu at (220.1, 69.7)
- added TP18: TestPoint_Probe, footprints:TestPoint_Hole_D1mm, F.Cu at (188.1, 66.1)
- added TP2: TestPoint_Probe, footprints:TestPoint_Hole_D1mm, F.Cu at (172.4, 135.7)
- added TP3: TestPoint_Probe, footprints:TestPoint_Hole_D1mm, F.Cu at (172.4, 137.7)
- added TP4: TestPoint_Probe, footprints:TestPoint_Hole_D1mm, F.Cu at (174.4, 133.7)
- added TP5: TestPoint_Probe, footprints:TestPoint_Hole_D1mm, F.Cu at (174.4, 135.7)
- added TP6: TestPoint_Probe, footprints:TestPoint_Hole_D1mm, F.Cu at (231.6, 126.8)
- added TP7: TestPoint_Probe, footprints:TestPoint_Hole_D1mm, F.Cu at (233.6, 122.8)
- added TP8: TestPoint_Probe, footprints:TestPoint_Hole_D1mm, F.Cu at (176.4, 135.7)
- added TP9: TestPoint_Probe, footprints:TestPoint_Hole_D1mm, F.Cu at (176.4, 137.7)
- added U1: AP7375-33SA-7, footprints:SOT-23-3_OEM, F.Cu at (248.1, 128.0)
- added U2: TCAN3413DR, footprints:SOIC-8_3.9x4.9mm_Pitch1.27mm_OEM, F.Cu at (249.8, 96.1)
- added Y1: 32_768kHz, footprints:XTAL_MU00525_NDK, F.Cu at (189.1, 124.2)
- added kibuzzard-670C7F9E: G***, kibuzzard-670C7F9E, F.Cu at (264.4, 86.5)
- added kibuzzard-670C854F: G***, kibuzzard-670C854F, F.Cu at (261.9, 86.5)
- added kibuzzard-670C8553: G***, kibuzzard-670C8553, F.Cu at (259.4, 86.5)
- added kibuzzard-670C8559: G***, kibuzzard-670C8559, F.Cu at (256.8, 86.5)
- added kibuzzard-670C856A: G***, kibuzzard-670C856A, F.Cu at (254.3, 86.5)
- added kibuzzard-670C856D: G***, kibuzzard-670C856D, F.Cu at (251.8, 86.5)
- added kibuzzard-670C8572: G***, kibuzzard-670C8572, F.Cu at (249.2, 86.5)
- added kibuzzard-670C8577: G***, kibuzzard-670C8577, F.Cu at (246.7, 86.5)
- added kibuzzard-670C857B: G***, kibuzzard-670C857B, F.Cu at (244.1, 86.5)
- added kibuzzard-670C8580: G***, kibuzzard-670C8580, F.Cu at (241.6, 86.5)
- added kibuzzard-670C8587: G***, kibuzzard-670C8587, F.Cu at (239.1, 86.5)
- added kibuzzard-670C85A1: G***, kibuzzard-670C85A1, F.Cu at (236.5, 86.5)
- added kibuzzard-670C85A5: G***, kibuzzard-670C85A5, F.Cu at (234.0, 86.5)
- added kibuzzard-670C8626: G***, kibuzzard-670C8626, F.Cu at (223.8, 86.5)
- added kibuzzard-670C8641: G***, kibuzzard-670C8641, F.Cu at (218.7, 86.5)
- added kibuzzard-670C864A: G***, kibuzzard-670C864A, F.Cu at (226.3, 86.5)
- added kibuzzard-670C864D: G***, kibuzzard-670C864D, F.Cu at (228.9, 86.5)
- added kibuzzard-670C8654: G***, kibuzzard-670C8654, F.Cu at (231.4, 86.5)
- added kibuzzard-670C865B: G***, kibuzzard-670C865B, F.Cu at (221.3, 86.5)
- added kibuzzard-670C8662: G***, kibuzzard-670C8662, F.Cu at (216.2, 86.5)
- added kibuzzard-670C866D: G***, kibuzzard-670C866D, F.Cu at (264.5, 100.8)
- added kibuzzard-670C8674: G***, kibuzzard-670C8674, F.Cu at (261.9, 100.8)
- added kibuzzard-670C8679: G***, kibuzzard-670C8679, F.Cu at (259.4, 100.8)
- added kibuzzard-670C8682: G***, kibuzzard-670C8682, F.Cu at (256.9, 100.8)
- added kibuzzard-670C8688: G***, kibuzzard-670C8688, F.Cu at (254.3, 100.8)
- added kibuzzard-670C8690: G***, kibuzzard-670C8690, F.Cu at (251.8, 100.8)
- added kibuzzard-670C8694: G***, kibuzzard-670C8694, F.Cu at (249.2, 100.8)
- added kibuzzard-670C8698: G***, kibuzzard-670C8698, F.Cu at (246.7, 100.8)
- added kibuzzard-670C86B2: G***, kibuzzard-670C86B2, F.Cu at (244.2, 100.8)
- added kibuzzard-670C86B8: G***, kibuzzard-670C86B8, F.Cu at (241.6, 100.8)
- added kibuzzard-670C86BC: G***, kibuzzard-670C86BC, F.Cu at (239.1, 100.8)
- added kibuzzard-670C86C0: G***, kibuzzard-670C86C0, F.Cu at (236.5, 100.8)
- added kibuzzard-670C86C5: G***, kibuzzard-670C86C5, F.Cu at (234.0, 100.8)
- added kibuzzard-670C86CA: G***, kibuzzard-670C86CA, F.Cu at (231.5, 100.8)
- added kibuzzard-670C86CE: G***, kibuzzard-670C86CE, F.Cu at (228.9, 100.8)
- added kibuzzard-670C86D3: G***, kibuzzard-670C86D3, F.Cu at (226.4, 100.8)
- added kibuzzard-670C86D7: G***, kibuzzard-670C86D7, F.Cu at (223.8, 100.8)
- added kibuzzard-670C86DC: G***, kibuzzard-670C86DC, F.Cu at (221.3, 100.8)
- added kibuzzard-670C86E5: G***, kibuzzard-670C86E5, F.Cu at (218.8, 100.8)
- added kibuzzard-670C86E9: G***, kibuzzard-670C86E9, F.Cu at (216.2, 100.8)
- C12: value C_4.7uF -> C_100nF
- C13: value C_100pF -> C_100nF
- C14: value C_100pF -> C_0.1uF
- C15: value C_1uF -> C_4.7uF
- C16, C17: value C_100nF -> C_100pF
- C4: value C_1uF -> C_5.1uF
- C5: value C_0.1uF -> C_10uF
- D10: value EAST16084WA1 -> ESDALC6V1W5; footprint footprints:WL-SMCD_0603 -> footprints:SOT323-5L
- D5: value USBLC6-2SC6 -> EAST16084WA1; footprint footprints:SOT-23-6_OEM -> footprints:WL-SMCD_0603
- D6: value SMAJ24A -> USBLC6-2SC6; footprint footprints:SMAJ24A-13-F -> footprints:SOT-23-6_OEM
- D7: value NUP2105LT1G -> SMAJ24A; footprint footprints:SOT-23-3_OEM -> footprints:SMAJ24A-13-F
- D8: value ESDALC6V1W5 -> NUP2105LT1G; footprint footprints:SOT323-5L -> footprints:SOT95P237X111-3N
- J5: value 2601-1104 -> 20p Header; footprint footprints:26011104 -> Connector_PinHeader_2.54mm:PinHeader_1x20_P2.54mm_Vertical; moved to B.Cu
- J6: value 2171790001 -> 20p Header; footprint footprints:MOLEX_2171790001 -> Connector_PinHeader_2.54mm:PinHeader_1x20_P2.54mm_Vertical; moved to B.Cu
- R10: value R_60.4 -> R_5.1k
- R12: value R_47 -> R_60.4
- R2, R3: value R_5.1k -> R_22
- R4: value R_10k -> R_47
- R8: value R_22 -> R_10k
- R9: value R_22 -> R_5.1k
- Y2: value 32KHz -> 24MHz; footprint footprints:Crystal_SMD_FA238 -> footprints:OSC_NX2016SA-24MHZ-EXS00A-CS10820
- moved J5 134.8 mm to (264.5, 102.5), turned to 90 degrees
- moved C16 130.4 mm to (263.1, 93.5), turned to 180 degrees
- moved C17 130.3 mm to (263.1, 98.5)
- moved C15 126.0 mm to (258.8, 96.0)
- moved R11 118.2 mm to (258.8, 94.5), turned to 180 degrees
- moved R12 118.2 mm to (258.8, 97.5)
- moved C14 117.1 mm to (245.2, 96.1), turned to 90 degrees
- moved D8 113.3 mm to (262.5, 96.0), turned to 180 degrees
- moved J6 108.0 mm to (264.5, 84.7), turned to 90 degrees
- moved FL1 105.8 mm to (255.5, 96.0)
- moved D5 101.7 mm to (237.2, 131.5)
- moved D2 91.1 mm to (228.6, 118.6)
- moved D9 87.8 mm to (232.6, 72.1)
- moved D10 82.7 mm to (235.2, 72.1)
- moved D1 64.0 mm to (223.0, 122.1)
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Connections:
- C11 pad 1: Net-(U3-Vin) -> +3V3
- C12 pad 1: Net-(C12-Pad1) -> /nRESET
- C13 pad 1: GND -> +3V3
- C13 pad 2: Net-(JP2-A) -> GND
- C14 pad 1: Net-(JP1-B) -> +3V3
- C15 pad 1: +3V3 -> Net-(C15-Pad1)
- C16 pad 1: +3V3 -> Net-(JP1-B)
- C17 pad 1: +3V3 -> GND
- C17 pad 2: GND -> Net-(JP2-A)
- C4 pad 1: +3V3 -> GND
- C4 pad 2: GND -> /OSC32_OUT
- D10 pad 1: GND -> /nRESET
- D10 pad 2: Net-(D10-Pad2) -> GND
- D2 pad 3: Net-(U3-Vin) -> Net-(U1-Vin)
- D5 pad 1: /DP_IN -> GND
- D5 pad 2: GND -> Net-(D5-Pad2)
- D6 pad 1: +VIN -> /DP_IN
- D7 pad 1: Net-(JP1-B) -> +VIN
- D7 pad 2: Net-(JP2-A) -> GND
- D8 pad 1: /NC/TDI -> Net-(JP2-A)
- D8 pad 2: GND -> Net-(JP1-B)
- D8 pad 3: /SWO/TDO -> GND
- D9 pad 1: /nRESET -> /NC/TDI
- D9 pad 3: /UART_TX -> /SWO/TDO
- D9 pad 4: /UART_RX -> /SWCLK/TCLK
- F1 pad 2: Net-(J6-VBUS1) -> Net-(J1-VBUS1)
- J5 pad 1: GND -> +VIN
- J5 pad 2: Net-(JP2-A) -> +VUSB
- J5 pad 3: Net-(JP1-B) -> +3V3
- J5 pad 4: +VUSB -> GND
- J5 pad 5: (no net) -> /PC13
- J5 pad 6: (no net) -> /PA0
- J5 pad 7: (no net) -> /PA1
- J5 pad 8: (no net) -> GND
- R10 pad 1: Net-(C12-Pad1) -> Net-(J1-CC2)
- R10 pad 2: Net-(JP2-A) -> GND
- R11 pad 2: Net-(C12-Pad1) -> Net-(C15-Pad1)
- R12 pad 1: /NC/TDI -> Net-(C15-Pad1)
- R12 pad 2: Net-(IC1-PA15) -> Net-(JP2-A)
- R2 pad 1: Net-(J6-CC2) -> Net-(IC1-PA11)
- R2 pad 2: GND -> /USB_DN
- R3 pad 1: Net-(J6-CC1) -> /USB_DP
- R3 pad 2: GND -> Net-(IC1-PA12)
- R4 pad 1: Net-(R4-Pad1) -> /NC/TDI
- R4 pad 2: /CAN_RX/BOOT -> Net-(IC1-PA15)
- R5 pad 1: +3V3 -> /PB14
- R5 pad 2: Net-(D1-Pad2) -> Net-(D3-Pad2)
- R8 pad 1: Net-(IC1-PA11) -> Net-(R8-Pad1)
- R8 pad 2: /USB_DN -> /CAN_RX/BOOT
- R9 pad 1: /USB_DP -> Net-(J1-CC1)
- R9 pad 2: Net-(IC1-PA12) -> GND
- Y2 pad 1: /OSC32_IN -> /OSC_IN
- Y2 pad 3: /OSC32_OUT -> /OSC_OUT

Commit message: continue layout
Parts:
- added C18: C_1uF, footprints:C_0603_1608Metric, F.Cu at (159.0, 104.2)
- added C19: C_100nF, footprints:C_0603_1608Metric, F.Cu at (159.0, 102.7)
- D1, D3, D4, D5: footprint footprints:WL-SMCD_0603 -> footprints:LED_0603_1608Metric
- D2: footprint footprints:SOT-23-3_OEM -> footprints:SOT95P237X111-3N
- J3: value MicroFit_V_2 -> PicoBlade; footprint footprints:MicroFit_V_2 -> footprints:CON_530480210_MOL
- JP1, JP2: moved to B.Cu
- U1: footprint footprints:SOT-23-3_OEM -> footprints:AP7375-33SA-7_DIO
- moved C10 110.4 mm to (142.9, 100.1)
- moved U1 109.6 mm to (142.9, 97.6), turned to -90 degrees
- moved J7 108.0 mm to (139.8, 103.2), turned to 90 degrees
- moved C9 107.6 mm to (142.9, 95.1)
- moved TP17 96.3 mm to (124.4, 80.7)
- moved R1 94.8 mm to (139.9, 117.6), turned to 90 degrees
- moved D2 92.0 mm to (139.0, 97.6)
- moved D5 83.4 mm to (154.1, 124.0)
- moved TP6 83.4 mm to (148.5, 119.2)
- moved TP7 83.4 mm to (150.5, 115.2)
- moved SW3 83.1 mm to (176.4, 93.0)
- moved D1 83.1 mm to (139.9, 120.6), turned to 90 degrees
- moved TP14 81.2 mm to (170.6, 92.0)
- moved TP15 81.2 mm to (167.2, 92.0)
- moved JP1 81.2 mm to (174.4, 96.7)
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Connections:
- U1 pad 2: GND -> +3V3
- U1 pad 3: (no net) -> GND
Other:
- board outline added: 78.2 x 22.9 mm

Commit message: place all components
Parts:
- added H1: 000_MOUNTING_HOLE, footprints:000_mounting_hole, F.Cu at (187.1, 87.7)
- added H2: 000_MOUNTING_HOLE, footprints:000_mounting_hole, F.Cu at (187.1, 107.2)
- added H3: 000_MOUNTING_HOLE, footprints:000_mounting_hole, F.Cu at (135.5, 103.3)
- added H4: 000_MOUNTING_HOLE, footprints:000_mounting_hole, F.Cu at (135.8, 92.2)
- moved TP17 71.1 mm to (190.4, 107.2)
- moved R6 56.8 mm to (166.9, 103.3), turned to -90 degrees
- moved D4 54.6 mm to (165.4, 103.3), turned to 90 degrees
- moved D3 53.1 mm to (163.9, 103.3), turned to 90 degrees
- moved R5 52.6 mm to (162.4, 103.3), turned to -90 degrees
- moved TP6 41.9 mm to (119.6, 88.9)
- moved TP7 39.2 mm to (121.4, 88.9)
- moved TP1 27.3 mm to (115.1, 90.9)
- moved TP10 27.3 mm to (121.1, 90.9)
- moved TP11 27.3 mm to (121.1, 92.9)
- moved TP12 27.3 mm to (121.1, 94.9)
- moved TP13 27.3 mm to (123.1, 90.9)
- moved TP2 27.3 mm to (115.1, 92.9)
- moved TP3 27.3 mm to (115.1, 94.9)
- moved TP4 27.3 mm to (117.1, 90.9)
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