File: vehicle/mkvii/hardware/bms/bms_core/bms_core.kicad_sch (KiCad schematic)
At the start: 32 parts, among them J1 CONN_02x03, J2 CONN_02x03, K1 Relay_G5Q-1A4-DC5, Q1 SSM3K333R, U1 ATMEGA64M1, U2 MAX33011EASA, Y1 Crystal_16MHz_18pF

Commit message: changed BMS Core
Parts:
- TP1, TP2: MPN 5019 -> 5010
Changed lines of the file:
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@@
 			)
 		)
-		(property "MPN" "5019"
+		(property "MPN" "5010"
 			(at 209.55 158.75 0)
 			(effects
@@
 			)
 		)
-		(property "MPN" "5019"
+		(property "MPN" "5010"
 			(at 209.55 153.67 0)
 			(effects

Commit message: FinalBMS
Parts:
- added H2: CONN_MountingHole, OEM:PCIe_Mount, symbol OEM:CONN_MountingHole
Connections:
- no-connect marks 9 -> 10
Changed lines of the file:
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@@
 	)
 	(no_connect
+		(at 196.85 151.13)
+	)
+	(no_connect
 		(at 41.91 53.34)
 	)
@@
 					(unit 1)
 				)
+			)
+		)
+	)
+	(symbol
+		(lib_id "OEM:CONN_MountingHole")
+		(at 196.85 148.59 0)
+		(unit 1)
+		(exclude_from_sim no)
+		(in_bom no)
+		(on_board yes)
+		(dnp no)
+		(fields_autoplaced yes)
+		(property "Reference" "H2"
+			(at 199.39 146.0499 0)
+			(effects
+				(font
+					(size 1.27 1.27)
+				)
+				(justify left)
+			)
+		)
+		(property "Value" "CONN_MountingHole"
+			(at 199.39 148.5899 0)
+			(effects
+				(font
+					(size 1.27 1.27)
+				)
+				(justify left)
+			)
+		)
+		(property "Footprint" "OEM:PCIe_Mount"
+			(at 196.85 148.59 0)
+			(effects
+				(font
+					(size 1.27 1.27)
+				)
+				(hide yes)
+			)
+		)
+		(property "Datasheet" "~"
+			(at 196.85 148.59 0)
+			(effects
+				(font
+					(size 1.27 1.27)
+				)
+				(hide yes)
+			)
+		)
+		(property "Description" "Mounting Hole with connection"
+			(at 196.85 148.59 0)
+			(effects
+				(font
+					(size 1.27 1.27)
+				)
+				(hide yes)
+			)
+		)
+		(pin "1"
+		)
+		(instances
+			(project ""
+				(path "/19b2a9f9-0be6-4bde-80c5-cbc5126d55d5"
+					(reference "H2")
+					(unit 1)
+				)
